File: pcb/robot/Charger.kicad_sch (KiCad schematic)
At the start: 27 parts, among them U13 MAX77976EFD+

Commit message: Modularized usb-pd board and main board split
Parts:
- renumbered NT5 to NT11, NT5 to NT6
