File: pcb/robot/Charger.kicad_sch (KiCad schematic)
At the start: 27 parts, among them U13 MAX77976EFD+

Commit message: Add removable I2C isolation jumpers on i2c0 and i2c1 (fixes #18)
Add a 0-ohm series resistor on both SDA and SCL for each slave on the
shared I2C buses, so a specific device can be isolated during
debugging (bus lockup / SDA-held-low) by pulling one resistor instead
of physical rework.

i2c0: R32/R33 (U1, STWLC38), R34/R35 (U12, fuel gauge), R36/R37 (U8,
motor driver), R38/R39 (U9, motor driver), R40/R53 (U6, MAX77857 -
placed between the level-shifter U5 and U6 so it isolates only that
branch). J9's existing link to the USB-PD module (R6/R7) was already
covered, no new jumper needed there.

i2c1: R55/R57 (U13, MAX77976 charger) and R65/R73 (J9's other I2C
link to the USB-PD module) - extended to this bus too, not just
i2c0 as the issue literally named, since the same lockup risk applies.

All 10 are 0-ohm, 0603, populated by default - only pull the one for
the suspect device during debugging. Placed for hand accessibility
where board space allowed.

Verified via ERC/DRC against the pre-#18 baseline: 0 unconnected
items, no new violations (318 ERC / 27 DRC, unchanged).

Co-Authored-By: Claude Sonnet 5 <noreply@anthropic.com>
Parts:
- added R55, R57: 0, robot:R_0603_1608Metric, symbol Device:R
Connections:
- net SCL: now also R55.1; no longer U13.24 (SCL)
- net SDA: now also R57.1; no longer U13.25 (SDA)
- new net: R55.2, U13.24 (SCL)
- new net: R57.2, U13.25 (SDA)
Changed lines of the file:
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@@
 	(text "Place D1 at edge of board. \n"
 		(exclude_from_sim no)
-		(at 83.185 127.635 0)
+		(at 65.786 130.048 0)
 		(effects
 			(font
@@
 	(wire
 		(pts
+			(xy 80.01 127) (xy 83.82 127)
+		)
+		(stroke
+			(width 0)
+			(type default)
+		)
+	)
+	(wire
+		(pts
 			(xy 86.36 137.16) (xy 96.52 137.16)
 		)
@@
 	(wire
 		(pts
-			(xy 64.77 137.16) (xy 68.58 137.16)
+			(xy 80.01 124.46) (xy 83.82 124.46)
 		)
 		(stroke
@@
 	(wire
 		(pts
-			(xy 243.84 109.22) (xy 264.16 109.22)
+			(xy 64.77 137.16) (xy 68.58 137.16)
 		)
 		(stroke
@@
 	(wire
 		(pts
-			(xy 83.82 104.14) (xy 92.71 104.14)
+			(xy 243.84 109.22) (xy 264.16 109.22)
 		)
 		(stroke
@@
 	(wire
 		(pts
-			(xy 69.85 121.92) (xy 96.52 121.92)
+			(xy 83.82 104.14) (xy 92.71 104.14)
 		)
 		(stroke
@@
 	(wire
 		(pts
-			(xy 92.71 96.52) (xy 96.52 96.52)
+			(xy 69.85 121.92) (xy 96.52 121.92)
 		)
 		(stroke
@@
 	(wire
 		(pts
-			(xy 264.16 109.22) (xy 271.78 109.22)
+			(xy 92.71 96.52) (xy 96.52 96.52)
 		)
 		(stroke
@@
 	(wire
 		(pts
-			(xy 193.04 106.68) (xy 193.04 109.22)
+			(xy 264.16 109.22) (xy 271.78 109.22)
 		)
 		(stroke
@@
 	(wire
 		(pts
-			(xy 264.16 99.06) (xy 271.78 99.06)
+			(xy 193.04 106.68) (xy 193.04 109.22)
 		)
 		(stroke
@@
 	(wire
 		(pts
-			(xy 92.71 127) (xy 96.52 127)
+			(xy 264.16 99.06) (xy 271.78 99.06)
 		)
 		(stroke
@@
 	(wire
 		(pts
-			(xy 92.71 124.46) (xy 96.52 124.46)
-		)
-		(stroke
-			(width 0)
-			(type default)
-		)
-	)
-	(wire
-		(pts
 			(xy 195.58 93.98) (xy 195.58 90.17)
 		)
@@
 	(wire
 		(pts
+			(xy 91.44 124.46) (xy 96.52 124.46)
+		)
+		(stroke
+			(width 0)
+			(type default)
+		)
+	)
+	(wire
+		(pts
 			(xy 17.78 81.28) (xy 17.78 82.55)
 		)
@@
 	(wire
 		(pts
+			(xy 91.44 127) (xy 96.52 127)
+		)
+		(stroke
+			(width 0)
+			(type default)
+		)
+	)
+	(wire
+		(pts
 			(xy 17.78 93.98) (xy 30.48 93.98)
 		)
@@
 	(hierarchical_label "SCL"
 		(shape input)
-		(at 92.71 124.46 180)
+		(at 80.01 124.46 180)
 		(effects
 			(font
@@
 	(hierarchical_label "SDA"
 		(shape input)
-		(at 92.71 127 180)
+		(at 80.01 127 180)
 		(effects
 			(font
@@
 					(unit 1)
 				)
+			)
+		)
+	)
+	(symbol
+		(lib_id "Device:R")
+		(at 87.63 124.46 90)
+		(unit 1)
+		(exclude_from_sim no)
+		(in_bom yes)
+		(on_board yes)
+		(dnp no)
+		(property "Reference" "R55"
+			(at 87.63 121.92 90)
+			(effects
+				(font
+					(size 1.27 1.27)
+				)
+			)
+		)
+		(property "Value" "0"
+			(at 87.63 124.46 90)
+			(effects
+				(font
+					(size 1.27 1.27)
+				)
+			)
+		)
+		(property "Footprint" "robot:R_0603_1608Metric"
+			(at 87.63 126.238 90)
+			(effects
+				(font
+					(size 1.27 1.27)
+				)
+				(hide yes)
+			)
+		)
+		(property "Datasheet" "~"
+			(at 87.63 124.46 0)
+			(effects
+				(font
+					(size 1.27 1.27)
+				)
+				(hide yes)
+			)
+		)
+		(property "Description" ""
+			(at 87.63 124.46 0)
+			(effects
+				(font
+					(size 1.27 1.27)
+				)
+			)
+		)
+		(property "Manufacturer" "Stackpole Electronics"
+			(at 87.63 124.46 90)
+			(effects
+				(font
+					(size 1.27 1.27)
+				)
+				(hide yes)
+			)
+		)
+		(property "Part Number" "RMCF0603ZT0R00"
+			(at 87.63 124.46 90)
+			(effects
+				(font
+					(size 1.27 1.27)
+				)
+				(hide yes)
+			)
+		)
+		(property "Stock" "15"
+			(at 87.63 124.46 0)
+			(effects
+				(font
+					(size 1.27 1.27)
+				)
+				(hide yes)
+			)
+		)
+		(property "Type" "SMD"
+			(at 87.63 124.46 0)
+			(effects
+				(font
+					(size 1.27 1.27)
+				)
+				(hide yes)
+			)
+		)
+		(pin "1"
+		)
+		(pin "2"
+		)
+		(instances
+			(project "robot"
+				(path "/0c7b298e-2d07-4b1f-b033-e95f02d45089/3b7e5198-fb12-4059-9002-c176f652e784"
+					(reference "R55")
+					(unit 1)
+				)
+			)
+		)
+	)
+	(symbol
+		(lib_id "Device:R")
+		(at 87.63 127 90)
+		(unit 1)
+		(exclude_from_sim no)
+		(in_bom yes)
+		(on_board yes)
+		(dnp no)
+		(property "Reference" "R57"
+			(at 82.296 128.27 90)
+			(effects
+				(font
+					(size 1.27 1.27)
+				)
+			)
+		)
+		(property "Value" "0"
+			(at 87.63 127 90)
+			(effects
+				(font
+					(size 1.27 1.27)
+				)
+			)
+		)
+		(property "Footprint" "robot:R_0603_1608Metric"
+			(at 87.63 128.778 90)
+			(effects
+				(font
+					(size 1.27 1.27)
+				)
+				(hide yes)
+			)
+		)
+		(property "Datasheet" "~"
+			(at 87.63 127 0)
+			(effects
+				(font
+					(size 1.27 1.27)
+				)
+				(hide yes)
+			)
+		)
+		(property "Description" ""
+			(at 87.63 127 0)
+			(effects
+				(font
+					(size 1.27 1.27)
+				)
+			)
+		)
+		(property "Manufacturer" "Stackpole Electronics"
+			(at 87.63 127 90)
+			(effects
+				(font
+					(size 1.27 1.27)
+				)
+				(hide yes)
+			)
+		)
+		(property "Part Number" "RMCF0603ZT0R00"
+			(at 87.63 127 90)
+			(effects
+				(font
+					(size 1.27 1.27)
+				)
+				(hide yes)
+			)
+		)
+		(property "Stock" "15"
+			(at 87.63 127 0)
+			(effects
+				(font
+					(size 1.27 1.27)
+				)
+				(hide yes)
+			)
+		)
+		(property "Type" "SMD"
+			(at 87.63 127 0)
+			(effects
+				(font
+					(size 1.27 1.27)
+				)
+				(hide yes)
+			)
+		)
+		(pin "1"
+		)
+		(pin "2"
+		)
+		(instances
+			(project "robot"
+				(path "/0c7b298e-2d07-4b1f-b033-e95f02d45089/3b7e5198-fb12-4059-9002-c176f652e784"
+					(reference "R57")
+					(unit 1)
+				)
