File: pcb/robot/Charger.kicad_sch (KiCad schematic)
At the start: 29 parts, among them U13 MAX77976EFD+

Commit message: Re-unify USB-PD module into main board (single-PCB architecture) (#17)
Merges the USB-PD module circuitry back into the main robot board as
a single PCB, reversing the earlier main-board/USB-PD-daughter-board
split. Full re-route and re-placement of the combined design:

- Consolidated low-profile parts toward the board center, using the
  space freed up by relocated capacitors, for better overall use of
  the available area.
- Kept all 0-ohm test/isolation jumpers in accessible locations for
  bench testing.
- Added/corrected footprints for several parts that had broken or
  incorrect footprints (DDC6_TEX variants, SOT-23-6, SOT-23-3,
  R0402).

Carries forward every closed correction issue and update made since
the original split: #3 (CC jumpers), #6 (IC1.ON pull-down), #14/#15
(ADC divider, motor connector pinout), #16, #18 (I2C isolation
jumpers), #19 (charger-sense GPIO interrupt), plus the BOM/pricing
updates, LED changes, and MAX77642 replacement.

Verified via kicad-cli ERC/DRC + netlist diff against the pre-merge
board: 0 unconnected items (unchanged), no new DRC error-level
violations besides one pre-existing excluded item, and the #6
(IC1.ON pull-down) and #19 (charger-sense GPIO interrupt) circuits
confirmed intact at the net-topology level despite the full-board
re-annotation changing most reference designators. Most of the raw
diff size is a KiCad 9 footprint-format upgrade (pre-2023 format
rewritten to current) rather than design changes - spot-checked
against unrelated footprints (e.g. mounting holes), which show
identical geometry under the new syntax.
Parts:
- NT18: renamed from NT6; symbol Device:NetTie_2 -> robot:NetTie_2
- NT19: renamed from NT11; symbol Device:NetTie_2 -> robot:NetTie_2
- NT21: renamed from NT5; symbol Device:NetTie_2 -> robot:NetTie_2
- R105: renamed from R55; symbol Device:R -> robot:R
- R106: renamed from R57; symbol Device:R -> robot:R
- renumbered C75 to C100, C76 to C101, C77 to C102, C78 to C105, C79 to C107, C80 to C108, C81 to C113, C82 to C116, C83 to C122, C67 to C61, C68 to C65, C69 to C68, C70 to C71, C71 to C75, C72 to C77, C73 to C90, D1 to D6, L2 to L5, R50 to R101, R56 to R103, R49 to R96, TP12 to TP30, U13 to U28
Changed lines of the file:
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@@
 		(dnp no)
 		(fields_autoplaced yes)
-		(property "Reference" "C75"
+		(property "Reference" "C100"
 			(at 187.96 125.7299 0)
 			(effects
@@
 			(project "robot"
 				(path "/0c7b298e-2d07-4b1f-b033-e95f02d45089/3b7e5198-fb12-4059-9002-c176f652e784"
-					(reference "C75")
+					(reference "C100")
 					(unit 1)
 				)
@@
 		(on_board yes)
 		(dnp no)
-		(property "Reference" "C72"
+		(property "Reference" "C77"
 			(at 88.9 97.7899 0)
 			(effects
@@
 			(project "robot"
 				(path "/0c7b298e-2d07-4b1f-b033-e95f02d45089/3b7e5198-fb12-4059-9002-c176f652e784"
-					(reference "C72")
+					(reference "C77")
 					(unit 1)
 				)
@@
 		(dnp no)
 		(fields_autoplaced yes)
-		(property "Reference" "R56"
+		(property "Reference" "R103"
 			(at 82.55 130.81 90)
 			(effects
@@
 			(project "robot"
 				(path "/0c7b298e-2d07-4b1f-b033-e95f02d45089/3b7e5198-fb12-4059-9002-c176f652e784"
-					(reference "R56")
+					(reference "R103")
 					(unit 1)
 				)
@@
 		(on_board yes)
 		(dnp no)
-		(property "Reference" "TP12"
+		(property "Reference" "TP30"
 			(at 50.8 160.02 0)
 			(effects
@@
 			(project "robot"
 				(path "/0c7b298e-2d07-4b1f-b033-e95f02d45089/3b7e5198-fb12-4059-9002-c176f652e784"
-					(reference "TP12")
+					(reference "TP30")
 					(unit 1)
 				)
@@
 		(on_board yes)
 		(dnp no)
-		(property "Reference" "C71"
+		(property "Reference" "C75"
 			(at 86.36 111.7599 0)
 			(effects
@@
 			(project "robot"
 				(path "/0c7b298e-2d07-4b1f-b033-e95f02d45089/3b7e5198-fb12-4059-9002-c176f652e784"
-					(reference "C71")
+					(reference "C75")
 					(unit 1)
 				)
@@
 		(dnp no)
 		(fields_autoplaced yes)
-		(property "Reference" "C68"
+		(property "Reference" "C65"
 			(at 34.29 83.8199 0)
 			(effects
@@
 			(project "robot"
 				(path "/0c7b298e-2d07-4b1f-b033-e95f02d45089/3b7e5198-fb12-4059-9002-c176f652e784"
-					(reference "C68")
+					(reference "C65")
 					(unit 1)
 				)
@@
 	)
 	(symbol
-		(lib_id "Device:NetTie_2")
+		(lib_id "robot:NetTie_2")
 		(at 62.23 137.16 0)
 		(unit 1)
@@
 		(on_board yes)
 		(dnp no)
-		(property "Reference" "NT11"
+		(property "Reference" "NT19"
 			(at 59.69 135.255 0)
 			(effects
@@
 			(project "robot"
 				(path "/0c7b298e-2d07-4b1f-b033-e95f02d45089/3b7e5198-fb12-4059-9002-c176f652e784"
-					(reference "NT11")
+					(reference "NT19")
 					(unit 1)
 				)
@@
 		(on_board yes)
 		(dnp no)
-		(property "Reference" "C81"
+		(property "Reference" "C113"
 			(at 220.98 100.3299 0)
 			(effects
@@
 			(project "robot"
 				(path "/0c7b298e-2d07-4b1f-b033-e95f02d45089/3b7e5198-fb12-4059-9002-c176f652e784"
-					(reference "C81")
+					(reference "C113")
 					(unit 1)
 				)
@@
 		(dnp no)
 		(fields_autoplaced yes)
-		(property "Reference" "D1"
+		(property "Reference" "D6"
 			(at 73.9775 129.54 0)
 			(effects
@@
 			(project "robot"
 				(path "/0c7b298e-2d07-4b1f-b033-e95f02d45089/3b7e5198-fb12-4059-9002-c176f652e784"
-					(reference "D1")
+					(reference "D6")
 					(unit 1)
 				)
@@
 		(on_board yes)
 		(dnp no)
-		(property "Reference" "C82"
+		(property "Reference" "C116"
 			(at 240.03 100.3299 0)
 			(effects
@@
 			(project "robot"
 				(path "/0c7b298e-2d07-4b1f-b033-e95f02d45089/3b7e5198-fb12-4059-9002-c176f652e784"
-					(reference "C82")
+					(reference "C116")
 					(unit 1)
 				)
@@
 		(on_board yes)
 		(dnp no)
-		(property "Reference" "C70"
+		(property "Reference" "C71"
 			(at 67.31 93.9799 0)
 			(effects
@@
 			(project "robot"
 				(path "/0c7b298e-2d07-4b1f-b033-e95f02d45089/3b7e5198-fb12-4059-9002-c176f652e784"
-					(reference "C70")
+					(reference "C71")
 					(unit 1)
 				)
@@
 		(on_board yes)
 		(dnp no)
-		(property "Reference" "C76"
+		(property "Reference" "C101"
 			(at 189.23 100.3299 0)
 			(effects
@@
 			(project "robot"
 				(path "/0c7b298e-2d07-4b1f-b033-e95f02d45089/3b7e5198-fb12-4059-9002-c176f652e784"
-					(reference "C76")
+					(reference "C101")
 					(unit 1)
 				)
@@
 		(dnp no)
 		(fields_autoplaced yes)
-		(property "Reference" "U13"
+		(property "Reference" "U28"
 			(at 121.8247 72.39 0)
 			(effects
@@
 			(project "robot"
 				(path "/0c7b298e-2d07-4b1f-b033-e95f02d45089/3b7e5198-fb12-4059-9002-c176f652e784"
-					(reference "U13")
+					(reference "U28")
 					(unit 1)
 				)
@@
 	)
 	(symbol
-		(lib_id "Device:NetTie_2")
+		(lib_id "robot:NetTie_2")
 		(at 27.305 163.83 0)
 		(unit 1)
@@
 		(on_board yes)
 		(dnp no)
-		(property "Reference" "NT6"
+		(property "Reference" "NT18"
 			(at 24.765 161.925 0)
 			(effects
@@
 			(project "robot"
 				(path "/0c7b298e-2d07-4b1f-b033-e95f02d45089/3b7e5198-fb12-4059-9002-c176f652e784"
-					(reference "NT6")
+					(reference "NT18")
 					(unit 1)
 				)
@@
 		(on_board yes)
 		(dnp no)
-		(property "Reference" "C83"
+		(property "Reference" "C122"
 			(at 260.35 100.3299 0)
 			(effects
@@
 			(project "robot"
 				(path "/0c7b298e-2d07-4b1f-b033-e95f02d45089/3b7e5198-fb12-4059-9002-c176f652e784"
-					(reference "C83")
+					(reference "C122")
 					(unit 1)
 				)
@@
 	)
 	(symbol
-		(lib_id "Device:NetTie_2")
+		(lib_id "robot:NetTie_2")
 		(at 226.06 129.54 270)
 		(unit 1)
@@
 		(on_board yes)
 		(dnp no)
-		(property "Reference" "NT5"
+		(property "Reference" "NT21"
 			(at 227.965 128.27 90)
 			(effects
@@
 			(project "robot"
 				(path "/0c7b298e-2d07-4b1f-b033-e95f02d45089/3b7e5198-fb12-4059-9002-c176f652e784"
-					(reference "NT5")
+					(reference "NT21")
 					(unit 1)
 				)
@@
 		(on_board yes)
 		(dnp no)
-		(property "Reference" "L2"
+		(property "Reference" "L5"
 			(at 171.45 92.71 0)
 			(effects
@@
 			(project "robot"
 				(path "/0c7b298e-2d07-4b1f-b033-e95f02d45089/3b7e5198-fb12-4059-9002-c176f652e784"
-					(reference "L2")
+					(reference "L5")
 					(unit 1)
 				)
@@
 		(on_board yes)
 		(dnp no)
-		(property "Reference" "C78"
+		(property "Reference" "C105"
 			(at 201.93 100.3299 0)
 			(effects
@@
 			(project "robot"
 				(path "/0c7b298e-2d07-4b1f-b033-e95f02d45089/3b7e5198-fb12-4059-9002-c176f652e784"
-					(reference "C78")
+					(reference "C105")
 					(unit 1)
 				)
@@
 		(dnp no)
 		(fields_autoplaced yes)
-		(property "Reference" "R49"
+		(property "Reference" "R96"
 			(at 72.39 113.0299 0)
 			(effects
@@
 			(project "robot"
 				(path "/0c7b298e-2d07-4b1f-b033-e95f02d45089/3b7e5198-fb12-4059-9002-c176f652e784"
-					(reference "R49")
+					(reference "R96")
 					(unit 1)
 				)
@@
 		(dnp no)
 		(fields_autoplaced yes)
-		(property "Reference" "C67"
+		(property "Reference" "C61"
 			(at 21.59 83.8199 0)
 			(effects
@@
 			(project "robot"
 				(path "/0c7b298e-2d07-4b1f-b033-e95f02d45089/3b7e5198-fb12-4059-9002-c176f652e784"
-					(reference "C67")
+					(reference "C61")
 					(unit 1)
 				)
@@
 		(dnp no)
 		(fields_autoplaced yes)
-		(property "Reference" "C80"
+		(property "Reference" "C108"
 			(at 212.09 83.8199 0)
 			(effects
@@
 			(project "robot"
 				(path "/0c7b298e-2d07-4b1f-b033-e95f02d45089/3b7e5198-fb12-4059-9002-c176f652e784"
-					(reference "C80")
+					(reference "C108")
 					(unit 1)
 				)
@@
 		(on_board yes)
 		(dnp no)
-		(property "Reference" "C69"
+		(property "Reference" "C68"
 			(at 54.61 93.9799 0)
 			(effects
@@
 			(project "robot"
 				(path "/0c7b298e-2d07-4b1f-b033-e95f02d45089/3b7e5198-fb12-4059-9002-c176f652e784"
-					(reference "C69")
+					(reference "C68")
 					(unit 1)
 				)
@@
 	)
 	(symbol
-		(lib_id "Device:R")
+		(lib_id "robot:R")
 		(at 87.63 124.46 90)
 		(unit 1)
@@
 		(on_board yes)
 		(dnp no)
-		(property "Reference" "R55"
+		(property "Reference" "R105"
 			(at 87.63 121.92 90)
 			(effects
@@
 			(project "robot"
 				(path "/0c7b298e-2d07-4b1f-b033-e95f02d45089/3b7e5198-fb12-4059-9002-c176f652e784"
-					(reference "R55")
+					(reference "R105")
 					(unit 1)
 				)
@@
 	)
 	(symbol
-		(lib_id "Device:R")
+		(lib_id "robot:R")
 		(at 87.63 127 90)
 		(unit 1)
@@
 		(on_board yes)
 		(dnp no)
-		(property "Reference" "R57"
+		(property "Reference" "R106"
 			(at 82.296 128.27 90)
 			(effects
@@
 			(project "robot"
 				(path "/0c7b298e-2d07-4b1f-b033-e95f02d45089/3b7e5198-fb12-4059-9002-c176f652e784"
-					(reference "R57")
+					(reference "R106")
 					(unit 1)
 				)
@@
 		(on_board yes)
 		(dnp no)
-		(property "Reference" "R50"
+		(property "Reference" "R101"
 			(at 72.39 148.59 90)
 			(effects
@@
 			(project "robot"
 				(path "/0c7b298e-2d07-4b1f-b033-e95f02d45089/3b7e5198-fb12-4059-9002-c176f652e784"
-					(reference "R50")
+					(reference "R101")
 					(unit 1)
 				)
@@
 		(dnp no)
 		(fields_autoplaced yes)
-		(property "Reference" "C77"
+		(property "Reference" "C102"
 			(at 191.77 83.8199 0)
 			(effects
@@
 			(project "robot"
 				(path "/0c7b298e-2d07-4b1f-b033-e95f02d45089/3b7e5198-fb12-4059-9002-c176f652e784"
-					(reference "C77")
+					(reference "C102")
 					(unit 1)
 				)
@@
 		(on_board yes)
 		(dnp yes)
-		(property "Reference" "C79"
+		(property "Reference" "C107"
 			(at 209.55 125.7299 0)
 			(effects
@@
 			(project "robot"
 				(path "/0c7b298e-2d07-4b1f-b033-e95f02d45089/3b7e5198-fb12-4059-9002-c176f652e784"
-					(reference "C79")
+					(reference "C107")
 					(unit 1)
 				)
@@
 		(on_board yes)
 		(dnp no)
-		(property "Reference" "C73"
+		(property "Reference" "C90"
 			(at 154.94 90.1699 0)
 			(effects
@@
 			(project "robot"
 				(path "/0c7b298e-2d07-4b1f-b033-e95f02d45089/3b7e5198-fb12-4059-9002-c176f652e784"
-					(reference "C73")
+					(reference "C90")
 					(unit 1)
 				)
