File: pcb/robot/LDO.kicad_sch (KiCad schematic)
At the start: 19 parts, among them U14 MAX77642ANA+

Commit message: Modularized usb-pd board and main board split
Parts:
- renumbered D1 to D2, R91 to R92, R91 to R93, R90 to R94
