File: pcb/robot/LDO.kicad_sch (KiCad schematic)
At the start: 15 parts, among them U10 TPS63021DSJR, U11 XC6206PxxxMR

Commit message: Re-unify USB-PD module into main board (single-PCB architecture) (#17)
Merges the USB-PD module circuitry back into the main robot board as
a single PCB, reversing the earlier main-board/USB-PD-daughter-board
split. Full re-route and re-placement of the combined design:

- Consolidated low-profile parts toward the board center, using the
  space freed up by relocated capacitors, for better overall use of
  the available area.
- Kept all 0-ohm test/isolation jumpers in accessible locations for
  bench testing.
- Added/corrected footprints for several parts that had broken or
  incorrect footprints (DDC6_TEX variants, SOT-23-6, SOT-23-3,
  R0402).

Carries forward every closed correction issue and update made since
the original split: #3 (CC jumpers), #6 (IC1.ON pull-down), #14/#15
(ADC divider, motor connector pinout), #16, #18 (I2C isolation
jumpers), #19 (charger-sense GPIO interrupt), plus the BOM/pricing
updates, LED changes, and MAX77642 replacement.

Verified via kicad-cli ERC/DRC + netlist diff against the pre-merge
board: 0 unconnected items (unchanged), no new DRC error-level
violations besides one pre-existing excluded item, and the #6
(IC1.ON pull-down) and #19 (charger-sense GPIO interrupt) circuits
confirmed intact at the net-topology level despite the full-board
re-annotation changing most reference designators. Most of the raw
diff size is a KiCad 9 footprint-format upgrade (pre-2023 format
rewritten to current) rather than design changes - spot-checked
against unrelated footprints (e.g. mounting holes), which show
identical geometry under the new syntax.
Parts:
- R28: renamed from R92; symbol Device:R -> robot:R
- R29: renamed from R94; symbol Device:R -> robot:R
- R30: renamed from R91; symbol Device:R -> robot:R
- U3: renamed from U11; symbol Regulator_Linear:XC6206PxxxMR -> robot:XC6206PxxxMR
- renumbered C4 to C2, C45 to C3, C92 to C4, C93 to C5, C94 to C6, C95 to C7, C46 to C8, C88 to C9, D2 to D1, L3 to L1, U10 to U2
Changed lines of the file:
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@@
 		(on_board yes)
 		(dnp no)
-		(property "Reference" "C93"
+		(property "Reference" "C5"
 			(at 121.92 71.1199 0)
 			(effects
@@
 			(project "robot"
 				(path "/0c7b298e-2d07-4b1f-b033-e95f02d45089/3b094808-5035-436e-9542-e9e286dde93f"
-					(reference "C93")
+					(reference "C5")
 					(unit 1)
 				)
@@
 		(on_board yes)
 		(dnp no)
-		(property "Reference" "C88"
+		(property "Reference" "C9"
 			(at 186.69 102.8699 0)
 			(effects
@@
 			(project "robot"
 				(path "/0c7b298e-2d07-4b1f-b033-e95f02d45089/3b094808-5035-436e-9542-e9e286dde93f"
-					(reference "C88")
+					(reference "C9")
 					(unit 1)
 				)
@@
 		(dnp no)
 		(fields_autoplaced yes)
-		(property "Reference" "D2"
+		(property "Reference" "D1"
 			(at 166.37 73.9775 0)
 			(effects
@@
 			(project "robot"
 				(path "/0c7b298e-2d07-4b1f-b033-e95f02d45089/3b094808-5035-436e-9542-e9e286dde93f"
-					(reference "D2")
+					(reference "D1")
 					(unit 1)
 				)
@@
 		(on_board yes)
 		(dnp no)
-		(property "Reference" "C92"
+		(property "Reference" "C4"
 			(at 50.8 78.7399 0)
 			(effects
@@
 			(project "robot"
 				(path "/0c7b298e-2d07-4b1f-b033-e95f02d45089/3b094808-5035-436e-9542-e9e286dde93f"
-					(reference "C92")
+					(reference "C4")
 					(unit 1)
 				)
@@
 		(dnp no)
 		(fields_autoplaced yes)
-		(property "Reference" "L3"
+		(property "Reference" "L1"
 			(at 119.38 85.0899 0)
 			(effects
@@
 			(project "robot"
 				(path "/0c7b298e-2d07-4b1f-b033-e95f02d45089/3b094808-5035-436e-9542-e9e286dde93f"
-					(reference "L3")
+					(reference "L1")
 					(unit 1)
 				)
@@
 	)
 	(symbol
-		(lib_id "Device:R")
+		(lib_id "robot:R")
 		(at 166.37 64.77 90)
 		(unit 1)
@@
 		(on_board yes)
 		(dnp no)
-		(property "Reference" "R94"
+		(property "Reference" "R29"
 			(at 166.37 62.23 90)
 			(effects
@@
 			(project "robot"
 				(path "/0c7b298e-2d07-4b1f-b033-e95f02d45089/3b094808-5035-436e-9542-e9e286dde93f"
-					(reference "R94")
+					(reference "R29")
 					(unit 1)
 				)
@@
 	)
 	(symbol
-		(lib_id "Regulator_Linear:XC6206PxxxMR")
+		(lib_id "robot:XC6206PxxxMR")
 		(at 173.99 101.6 0)
 		(unit 1)
@@
 		(on_board yes)
 		(dnp no)
-		(property "Reference" "U11"
+		(property "Reference" "U3"
 			(at 173.99 95.25 0)
 			(effects
@@
 			(project ""
 				(path "/0c7b298e-2d07-4b1f-b033-e95f02d45089/3b094808-5035-436e-9542-e9e286dde93f"
-					(reference "U11")
+					(reference "U3")
 					(unit 1)
 				)
@@
 		(on_board yes)
 		(dnp no)
-		(property "Reference" "C45"
+		(property "Reference" "C3"
 			(at 39.37 67.31 0)
 			(effects
@@
 			(project "robot"
 				(path "/0c7b298e-2d07-4b1f-b033-e95f02d45089/3b094808-5035-436e-9542-e9e286dde93f"
-					(reference "C45")
+					(reference "C3")
 					(unit 1)
 				)
@@
 		(on_board yes)
 		(dnp no)
-		(property "Reference" "C46"
+		(property "Reference" "C8"
 			(at 160.02 102.8699 0)
 			(effects
@@
 			(project "robot"
 				(path "/0c7b298e-2d07-4b1f-b033-e95f02d45089/3b094808-5035-436e-9542-e9e286dde93f"
-					(reference "C46")
+					(reference "C8")
 					(unit 1)
 				)
@@
 		(on_board yes)
 		(dnp no)
-		(property "Reference" "C4"
+		(property "Reference" "C2"
 			(at 26.67 67.31 0)
 			(effects
@@
 			(project "robot"
 				(path "/0c7b298e-2d07-4b1f-b033-e95f02d45089/3b094808-5035-436e-9542-e9e286dde93f"
-					(reference "C4")
+					(reference "C2")
 					(unit 1)
 				)
@@
 		(on_board yes)
 		(dnp no)
-		(property "Reference" "C94"
+		(property "Reference" "C6"
 			(at 133.35 71.1199 0)
 			(effects
@@
 			(project "robot"
 				(path "/0c7b298e-2d07-4b1f-b033-e95f02d45089/3b094808-5035-436e-9542-e9e286dde93f"
-					(reference "C94")
+					(reference "C6")
 					(unit 1)
 				)
@@
 	)
 	(symbol
-		(lib_id "Device:R")
+		(lib_id "robot:R")
 		(at 68.58 77.47 90)
 		(unit 1)
@@
 		(on_board yes)
 		(dnp no)
-		(property "Reference" "R92"
+		(property "Reference" "R28"
 			(at 68.58 74.93 90)
 			(effects
@@
 			(project "robot"
 				(path "/0c7b298e-2d07-4b1f-b033-e95f02d45089/3b094808-5035-436e-9542-e9e286dde93f"
-					(reference "R92")
+					(reference "R28")
 					(unit 1)
 				)
@@
 	)
 	(symbol
-		(lib_id "Device:R")
+		(lib_id "robot:R")
 		(at 196.85 101.6 90)
 		(unit 1)
@@
 		(on_board yes)
 		(dnp no)
-		(property "Reference" "R91"
+		(property "Reference" "R30"
 			(at 196.85 99.06 90)
 			(effects
@@
 			(project "robot"
 				(path "/0c7b298e-2d07-4b1f-b033-e95f02d45089/3b094808-5035-436e-9542-e9e286dde93f"
-					(reference "R91")
+					(reference "R30")
 					(unit 1)
 				)
@@
 		(on_board yes)
 		(dnp no)
-		(property "Reference" "C95"
+		(property "Reference" "C7"
 			(at 143.51 71.1199 0)
 			(effects
@@
 			(project "robot"
 				(path "/0c7b298e-2d07-4b1f-b033-e95f02d45089/3b094808-5035-436e-9542-e9e286dde93f"
-					(reference "C95")
+					(reference "C7")
 					(unit 1)
 				)
@@
 		(dnp no)
 		(fields_autoplaced yes)
-		(property "Reference" "U10"
+		(property "Reference" "U2"
 			(at 92.71 57.15 0)
 			(effects
@@
 			(project ""
 				(path "/0c7b298e-2d07-4b1f-b033-e95f02d45089/3b094808-5035-436e-9542-e9e286dde93f"
-					(reference "U10")
+					(reference "U2")
 					(unit 1)
 				)
