File: pcb/robot/Protection.kicad_sch (KiCad schematic)
At the start: 44 parts, among them IC1 TPS22998RYZR, Q1 Q_NMOS_GDS, Q2 EFC8811R-TF, SW1 SW_SPST, U12 BQ27742YZFR-G1

Commit message: Modularized usb-pd board and main board split
Parts:
- renumbered D1 to D3, NT5 to NT10, NT5 to NT12, NT5 to NT13, NT5 to NT7, NT5 to NT8, NT5 to NT9, Q1 to Q7, R18 to R8
