File: pcb/robot/Protection.kicad_sch (KiCad schematic)
At the start: 44 parts, among them IC1 TPS22998RYZR, Q2 EFC8811R-TF, Q7 Q_NMOS_GDS, SW1 SW_SPST, U12 BQ27742YZFR-G1

Commit message: Fix reversed motor connector pins on J3/J5 (fixes #15)
Swap pins 1/6 (motor phase polarity) and 2/5 (encoder VCC/GND) on
both motor JST connectors (J3, J5), so standard JST cables work
without custom re-pinning and without needing a software-side
forward/backward negation workaround. Pins 3/4 (encoder A/B) left
untouched. PCB copper re-routed to match; verified 0 unconnected
items via DRC and no new ERC violations on J3/J5.

Firmware's negation workaround should be removed once this hardware
revision is in use, or the two corrections will cancel out.

Fix leftover note typo and grid nudge (follow-up to #3)

Correct CC jumper note in USB_PD_Module.kicad_sch to reference the
actual R3/R4 designators used, and nudge SW1 onto grid in
Protection.kicad_sch. No net changes.
Other:
- moved on the sheet: SW1
Changed lines of the file:
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@@
 	(wire
 		(pts
-			(xy 327.025 110.49) (xy 315.595 110.49)
+			(xy 327.66 110.49) (xy 315.595 110.49)
 		)
 		(stroke
@@
 	(wire
 		(pts
-			(xy 327.025 91.44) (xy 332.105 91.44)
+			(xy 327.66 91.44) (xy 332.105 91.44)
 		)
 		(stroke
@@
 	(wire
 		(pts
-			(xy 327.025 93.98) (xy 327.025 110.49)
+			(xy 327.66 93.98) (xy 327.66 110.49)
 		)
 		(stroke
@@
 	(wire
 		(pts
-			(xy 315.595 91.44) (xy 316.865 91.44)
+			(xy 315.595 91.44) (xy 317.5 91.44)
 		)
 		(stroke
@@
 	(symbol
 		(lib_id "robot:SW_SPST_S1S2pins")
-		(at 321.945 91.44 0)
+		(at 322.58 91.44 0)
 		(unit 1)
 		(exclude_from_sim no)
@@
 		(dnp no)
 		(property "Reference" "SW1"
-			(at 321.945 85.09 0)
+			(at 322.58 85.09 0)
 			(effects
 				(font
@@
 		)
 		(property "Value" "SW_SPST"
-			(at 321.945 87.63 0)
+			(at 322.58 87.63 0)
 			(effects
 				(font
@@
 		)
 		(property "Footprint" "robot:MOLEX_picoblade_SMT_2pin"
-			(at 321.945 97.79 0)
+			(at 322.58 97.79 0)
 			(effects
 				(font
@@
 		)
 		(property "Datasheet" "https://tools.molex.com/pdm_docs/sd/533980271_sd.pdf"
-			(at 321.945 99.06 0)
+			(at 322.58 99.06 0)
 			(effects
 				(font
@@
 		)
 		(property "Description" ""
-			(at 321.945 91.44 0)
+			(at 322.58 91.44 0)
 			(effects
 				(font
@@
 		)
 		(property "Manufacturer" "Molex"
-			(at 321.945 96.52 0)
+			(at 322.58 96.52 0)
 			(effects
 				(font
@@
 		)
 		(property "Part Number" "0533980271"
-			(at 321.945 97.79 0)
+			(at 322.58 97.79 0)
 			(effects
 				(font
@@
 		)
 		(property "Stock" ""
-			(at 321.945 91.44 0)
+			(at 322.58 91.44 0)
 			(effects
 				(font
@@
 		)
 		(property "Type" "SMD"
-			(at 321.945 91.44 0)
+			(at 322.58 91.44 0)
 			(effects
 				(font

Commit message: Add 470k pull-down on IC1.ON to fix floating pin when off (fixes #6)
Replace DNP C99 (1uF cap) with populated R13 (470kOhm, LCSC C25562) from IC1.ON to GND - was floating when SW1 is open. Sized per TPS22998 worst-case (falling threshold min 0.595V, leakage max 1uA). Verified via ERC/DRC against baseline: no regressions, 0 unconnected items before/after.
Parts:
- removed C99: 1uF, robot:C_0402_1005Metric, symbol robot:C
- added R13: 0402WGJ0474TCE, easyeda2kicad:R0402, symbol easyeda2kicad:0402WGJ0474TCE
Connections:
- net PGND: now also R13.2
- net at IC1.10 (ON), SW1.1 (A): now also R13.1
Changed lines of the file:
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@@
 	)
 	(junction
-		(at 315.595 91.44)
-		(diameter 0)
-		(color 0 0 0 0)
-	)
-	(junction
 		(at 180.34 168.91)
 		(diameter 0)
@@
 	)
 	(junction
-		(at 315.595 110.49)
+		(at 170.815 118.11)
 		(diameter 0)
 		(color 0 0 0 0)
 	)
 	(junction
-		(at 170.815 118.11)
+		(at 170.815 105.41)
 		(diameter 0)
 		(color 0 0 0 0)
 	)
 	(junction
-		(at 170.815 105.41)
+		(at 316.23 91.44)
 		(diameter 0)
 		(color 0 0 0 0)
@@
 	)
 	(junction
+		(at 316.23 110.49)
+		(diameter 0)
+		(color 0 0 0 0)
+	)
+	(junction
 		(at 99.06 156.21)
 		(diameter 0)
@@
 	(wire
 		(pts
-			(xy 315.595 107.95) (xy 315.595 110.49)
-		)
-		(stroke
-			(width 0)
-			(type default)
-		)
-	)
-	(wire
-		(pts
 			(xy 190.5 81.28) (xy 190.5 78.74)
 		)
@@
 	(wire
 		(pts
-			(xy 315.595 91.44) (xy 315.595 100.33)
+			(xy 365.125 198.12) (xy 410.21 198.12)
 		)
 		(stroke
@@
 	(wire
 		(pts
-			(xy 365.125 198.12) (xy 410.21 198.12)
+			(xy 50.8 147.32) (xy 50.8 135.89)
 		)
 		(stroke
@@
 	(wire
 		(pts
-			(xy 50.8 147.32) (xy 50.8 135.89)
+			(xy 90.17 168.91) (xy 90.17 148.59)
 		)
 		(stroke
@@
 	(wire
 		(pts
-			(xy 90.17 168.91) (xy 90.17 148.59)
+			(xy 227.965 88.265) (xy 227.965 109.22)
 		)
 		(stroke
@@
 	(wire
 		(pts
-			(xy 227.965 88.265) (xy 227.965 109.22)
+			(xy 155.575 93.98) (xy 160.655 93.98)
 		)
 		(stroke
@@
 	(wire
 		(pts
-			(xy 155.575 93.98) (xy 160.655 93.98)
+			(xy 316.23 91.44) (xy 316.23 96.52)
 		)
 		(stroke
@@
 	(wire
 		(pts
-			(xy 327.66 110.49) (xy 315.595 110.49)
-		)
-		(stroke
-			(width 0)
-			(type default)
-		)
-	)
-	(wire
-		(pts
 			(xy 248.92 81.28) (xy 264.16 81.28)
 		)
@@
 	(wire
 		(pts
+			(xy 316.23 110.49) (xy 327.66 110.49)
+		)
+		(stroke
+			(width 0)
+			(type default)
+		)
+	)
+	(wire
+		(pts
 			(xy 340.995 198.12) (xy 352.425 198.12)
 		)
@@
 	(wire
 		(pts
+			(xy 316.23 91.44) (xy 317.5 91.44)
+		)
+		(stroke
+			(width 0)
+			(type default)
+		)
+	)
+	(wire
+		(pts
 			(xy 43.18 114.3) (xy 43.18 133.35)
 		)
@@
 	(wire
 		(pts
-			(xy 282.575 110.49) (xy 315.595 110.49)
+			(xy 316.23 106.68) (xy 316.23 110.49)
+		)
+		(stroke
+			(width 0)
+			(type default)
+		)
+	)
+	(wire
+		(pts
+			(xy 282.575 110.49) (xy 316.23 110.49)
 		)
 		(stroke
@@
 	(wire
 		(pts
-			(xy 315.595 91.44) (xy 317.5 91.44)
+			(xy 315.595 91.44) (xy 316.23 91.44)
 		)
 		(stroke
@@
 	(symbol
 		(lib_id "robot:C")
-		(at 315.595 104.14 0)
-		(unit 1)
-		(exclude_from_sim no)
-		(in_bom yes)
-		(on_board yes)
-		(dnp yes)
-		(property "Reference" "C99"
-			(at 319.405 102.8699 0)
-			(effects
-				(font
-					(size 1.27 1.27)
-				)
-				(justify left)
-			)
-		)
-		(property "Value" "1uF"
-			(at 319.405 105.4099 0)
-			(effects
-				(font
-					(size 1.27 1.27)
-				)
-				(justify left)
-			)
-		)
-		(property "Footprint" "robot:C_0402_1005Metric"
-			(at 316.5602 107.95 0)
-			(effects
-				(font
-					(size 1.27 1.27)
-				)
-				(hide yes)
-			)
-		)
-		(property "Datasheet" "~"
-			(at 315.595 104.14 0)
-			(effects
-				(font
-					(size 1.27 1.27)
-				)
-				(hide yes)
-			)
-		)
-		(property "Description" "10V"
-			(at 321.945 107.95 0)
-			(effects
-				(font
-					(size 1.27 1.27)
-				)
-			)
-		)
-		(property "Manufacturer" "Murata"
-			(at 315.595 104.14 0)
-			(effects
-				(font
-					(size 1.27 1.27)
-				)
-				(hide yes)
-			)
-		)
-		(property "Part Number" "GRM155R61E105KA12D"
-			(at 315.595 104.14 0)
-			(effects
-				(font
-					(size 1.27 1.27)
-				)
-				(hide yes)
-			)
-		)
-		(property "Stock" "10"
-			(at 315.595 104.14 0)
-			(effects
-				(font
-					(size 1.27 1.27)
-				)
-				(hide yes)
-			)
-		)
-		(property "Type" "SMD"
-			(at 315.595 104.14 0)
-			(effects
-				(font
-					(size 1.27 1.27)
-				)
-				(hide yes)
-			)
-		)
-		(pin "1"
-		)
-		(pin "2"
-		)
-		(instances
-			(project "robot"
-				(path "/0c7b298e-2d07-4b1f-b033-e95f02d45089/aaf20b87-68dc-43c9-a7d3-4ceda8b87424"
-					(reference "C99")
-					(unit 1)
-				)
-			)
-		)
-	)
-	(symbol
-		(lib_id "robot:C")
 		(at 214.63 69.85 90)
 		(unit 1)
@@
 					(unit 1)
 				)
+			)
+		)
+	)
+	(symbol
+		(lib_id "easyeda2kicad:0402WGJ0474TCE")
+		(at 316.23 101.6 270)
+		(unit 1)
+		(exclude_from_sim no)
+		(in_bom yes)
+		(on_board yes)
+		(dnp no)
+		(property "Reference" "R13"
+			(at 319.278 101.6 0)
+			(effects
+				(font
+					(size 1.27 1.27)
+				)
+			)
+		)
+		(property "Value" "0402WGJ0474TCE"
+			(at 320.04 101.6 0)
+			(effects
+				(font
+					(size 1.27 1.27)
+				)
+				(hide yes)
+			)
+		)
+		(property "Footprint" "easyeda2kicad:R0402"
+			(at 308.61 101.6 0)
+			(effects
+				(font
+					(size 1.27 1.27)
+				)
+				(hide yes)
+			)
+		)
+		(property "Datasheet" "https://lcsc.com/product-detail/Chip-Resistor-Surface-Mount-UniOhm_470KR-474-5_C25562.html"
+			(at 306.07 101.6 0)
+			(effects
+				(font
+					(size 1.27 1.27)
+				)
+				(hide yes)
+			)
+		)
+		(property "Description" "470KΩ"
+			(at 313.944 101.092 0)
+			(effects
+				(font
+					(size 1.27 1.27)
+				)
+			)
+		)
+		(property "Manufacturer" "UNI-ROYAL(厚声)"
+			(at 303.53 101.6 0)
+			(effects
+				(font
+					(size 1.27 1.27)
+				)
+				(hide yes)
+			)
+		)
+		(property "MPN" "0402WGJ0474TCE"
+			(at 300.99 101.6 0)
+			(effects
+				(font
+					(size 1.27 1.27)
+				)
+				(hide yes)
+			)
+		)
+		(property "LCSC Part" "C25562"
+			(at 298.45 101.6 0)
+			(effects
+				(font
+					(size 1.27 1.27)
+				)
+				(hide yes)
+			)
+		)
+		(property "Part Number" "0402WGJ0474TCE"
+			(at 316.23 101.6 0)
+			(effects
+				(font
+					(size 1.27 1.27)
+				)
+				(hide yes)
+			)
+		)
+		(pin "2"
+		)
+		(pin "1"
+		)
+		(instances
+			(project ""
+				(path "/0c7b298e-2d07-4b1f-b033-e95f02d45089/aaf20b87-68dc-43c9-a7d3-4ceda8b87424"
+					(reference "R13")
+					(unit 1)
+				)
