File: pcb/robot/Protection.kicad_sch (KiCad schematic)
At the start: 44 parts, among them IC1 TPS22998RYZR, Q2 EFC8811R-TF, Q7 Q_NMOS_GDS, SW1 SW_SPST, U12 BQ27742YZFR-G1

Commit message: Add removable I2C isolation jumpers on i2c0 and i2c1 (fixes #18)
Add a 0-ohm series resistor on both SDA and SCL for each slave on the
shared I2C buses, so a specific device can be isolated during
debugging (bus lockup / SDA-held-low) by pulling one resistor instead
of physical rework.

i2c0: R32/R33 (U1, STWLC38), R34/R35 (U12, fuel gauge), R36/R37 (U8,
motor driver), R38/R39 (U9, motor driver), R40/R53 (U6, MAX77857 -
placed between the level-shifter U5 and U6 so it isolates only that
branch). J9's existing link to the USB-PD module (R6/R7) was already
covered, no new jumper needed there.

i2c1: R55/R57 (U13, MAX77976 charger) and R65/R73 (J9's other I2C
link to the USB-PD module) - extended to this bus too, not just
i2c0 as the issue literally named, since the same lockup risk applies.

All 10 are 0-ohm, 0603, populated by default - only pull the one for
the suspect device during debugging. Placed for hand accessibility
where board space allowed.

Verified via ERC/DRC against the pre-#18 baseline: 0 unconnected
items, no new violations (318 ERC / 27 DRC, unchanged).

Co-Authored-By: Claude Sonnet 5 <noreply@anthropic.com>
Parts:
- added R34, R35: 0, robot:R_0603_1608Metric, symbol Device:R
Connections:
- net SCL: now also R34.2; no longer U12.E3 (SCL)
- net SDA: now also R35.2; no longer U12.C3 (SDA)
- new net: R34.1, U12.E3 (SCL)
- new net: R35.1, U12.C3 (SDA)
Changed lines of the file:
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@@
 	(wire
 		(pts
+			(xy 151.13 156.21) (xy 154.94 156.21)
+		)
+		(stroke
+			(width 0)
+			(type default)
+		)
+	)
+	(wire
+		(pts
+			(xy 151.13 153.67) (xy 154.94 153.67)
+		)
+		(stroke
+			(width 0)
+			(type default)
+		)
+	)
+	(wire
+		(pts
 			(xy 315.595 81.28) (xy 315.595 83.82)
 		)
@@
 	(wire
 		(pts
+			(xy 140.97 156.21) (xy 143.51 156.21)
+		)
+		(stroke
+			(width 0)
+			(type default)
+		)
+	)
+	(wire
+		(pts
 			(xy 264.16 198.12) (xy 340.995 198.12)
 		)
@@
 	(wire
 		(pts
-			(xy 248.92 81.28) (xy 264.16 81.28)
+			(xy 140.97 153.67) (xy 143.51 153.67)
 		)
 		(stroke
@@
 	(wire
 		(pts
-			(xy 190.5 69.85) (xy 195.58 69.85)
+			(xy 248.92 81.28) (xy 264.16 81.28)
 		)
 		(stroke
@@
 	(wire
 		(pts
-			(xy 170.815 105.41) (xy 170.815 118.11)
+			(xy 190.5 69.85) (xy 195.58 69.85)
 		)
 		(stroke
@@
 	(wire
 		(pts
-			(xy 140.97 153.67) (xy 158.75 153.67)
+			(xy 170.815 105.41) (xy 170.815 118.11)
 		)
 		(stroke
@@
 	(wire
 		(pts
-			(xy 140.97 156.21) (xy 158.75 156.21)
-		)
-		(stroke
-			(width 0)
-			(type default)
-		)
-	)
-	(wire
-		(pts
 			(xy 43.18 198.12) (xy 248.92 198.12)
 		)
@@
 	(hierarchical_label "SCL"
 		(shape input)
-		(at 158.75 153.67 0)
+		(at 154.94 153.67 0)
 		(effects
 			(font
@@
 	(hierarchical_label "SDA"
 		(shape input)
-		(at 158.75 156.21 0)
+		(at 154.94 156.21 0)
 		(effects
 			(font
@@
 	)
 	(symbol
+		(lib_id "Device:R")
+		(at 147.32 153.67 90)
+		(unit 1)
+		(exclude_from_sim no)
+		(in_bom yes)
+		(on_board yes)
+		(dnp no)
+		(property "Reference" "R34"
+			(at 147.32 151.13 90)
+			(effects
+				(font
+					(size 1.27 1.27)
+				)
+			)
+		)
+		(property "Value" "0"
+			(at 147.32 153.67 90)
+			(effects
+				(font
+					(size 1.27 1.27)
+				)
+			)
+		)
+		(property "Footprint" "robot:R_0603_1608Metric"
+			(at 147.32 155.448 90)
+			(effects
+				(font
+					(size 1.27 1.27)
+				)
+				(hide yes)
+			)
+		)
+		(property "Datasheet" "~"
+			(at 147.32 153.67 0)
+			(effects
+				(font
+					(size 1.27 1.27)
+				)
+				(hide yes)
+			)
+		)
+		(property "Description" ""
+			(at 147.32 153.67 0)
+			(effects
+				(font
+					(size 1.27 1.27)
+				)
+			)
+		)
+		(property "Manufacturer" "Stackpole Electronics"
+			(at 147.32 153.67 90)
+			(effects
+				(font
+					(size 1.27 1.27)
+				)
+				(hide yes)
+			)
+		)
+		(property "Part Number" "RMCF0603ZT0R00"
+			(at 147.32 153.67 90)
+			(effects
+				(font
+					(size 1.27 1.27)
+				)
+				(hide yes)
+			)
+		)
+		(property "Stock" "15"
+			(at 147.32 153.67 0)
+			(effects
+				(font
+					(size 1.27 1.27)
+				)
+				(hide yes)
+			)
+		)
+		(property "Type" "SMD"
+			(at 147.32 153.67 0)
+			(effects
+				(font
+					(size 1.27 1.27)
+				)
+				(hide yes)
+			)
+		)
+		(pin "1"
+		)
+		(pin "2"
+		)
+		(instances
+			(project "robot"
+				(path "/0c7b298e-2d07-4b1f-b033-e95f02d45089/aaf20b87-68dc-43c9-a7d3-4ceda8b87424"
+					(reference "R34")
+					(unit 1)
+				)
+			)
+		)
+	)
+	(symbol
 		(lib_id "robot:Q_NMOS_GSD")
 		(at 177.8 176.53 0)
@@
 					(unit 1)
 				)
+			)
+		)
+	)
+	(symbol
+		(lib_id "Device:R")
+		(at 147.32 156.21 90)
+		(unit 1)
+		(exclude_from_sim no)
+		(in_bom yes)
+		(on_board yes)
+		(dnp no)
+		(property "Reference" "R35"
+			(at 147.32 158.496 90)
+			(effects
+				(font
+					(size 1.27 1.27)
+				)
+			)
+		)
+		(property "Value" "0"
+			(at 147.32 156.21 90)
+			(effects
+				(font
+					(size 1.27 1.27)
+				)
+			)
+		)
+		(property "Footprint" "robot:R_0603_1608Metric"
+			(at 147.32 157.988 90)
+			(effects
+				(font
+					(size 1.27 1.27)
+				)
+				(hide yes)
+			)
+		)
+		(property "Datasheet" "~"
+			(at 147.32 156.21 0)
+			(effects
+				(font
+					(size 1.27 1.27)
+				)
+				(hide yes)
+			)
+		)
+		(property "Description" ""
+			(at 147.32 156.21 0)
+			(effects
+				(font
+					(size 1.27 1.27)
+				)
+			)
+		)
+		(property "Manufacturer" "Stackpole Electronics"
+			(at 147.32 156.21 90)
+			(effects
+				(font
+					(size 1.27 1.27)
+				)
+				(hide yes)
+			)
+		)
+		(property "Part Number" "RMCF0603ZT0R00"
+			(at 147.32 156.21 90)
+			(effects
+				(font
+					(size 1.27 1.27)
+				)
+				(hide yes)
+			)
+		)
+		(property "Stock" "15"
+			(at 147.32 156.21 0)
+			(effects
+				(font
+					(size 1.27 1.27)
+				)
+				(hide yes)
+			)
+		)
+		(property "Type" "SMD"
+			(at 147.32 156.21 0)
+			(effects
+				(font
+					(size 1.27 1.27)
+				)
+				(hide yes)
+			)
+		)
+		(pin "1"
+		)
+		(pin "2"
+		)
+		(instances
+			(project "robot"
+				(path "/0c7b298e-2d07-4b1f-b033-e95f02d45089/aaf20b87-68dc-43c9-a7d3-4ceda8b87424"
+					(reference "R35")
+					(unit 1)
+				)
