File: pcb/robot/USB-PD-PhonePC.kicad_sch (KiCad schematic)
At the start: 54 parts, among them J4 USB4151-GF-C, U11 MAX77958EWV+T, U15 TPD1E05U06, U16 fpf1048bucx, U17 TPS61253AYFFT, U19 TPD1E05U06, U20 TPD1E05U06, U21 TPD1E05U06, U22 TPD1E05U06, U23 TPD1E05U06, U24 TVS0500DRV

Commit message: Modularized usb-pd board and main board split
Parts:
- removed C100, C101, C97: 4.7uF, robot:C_0603_1608Metric, symbol robot:C
- removed C45, C46: 27pF, robot:C_0402_1005Metric, symbol robot:C
- removed C47, C48, C50, C51, C52, C53, C54: 1uF, robot:C_0402_1005Metric, symbol robot:C
- removed C49: 2.2uF, robot:C_0603_1608Metric, symbol robot:C
- removed J4: USB4151-GF-C, robot:GCT_USB4151-GF-C_REVA, symbol robot:USB4151-GF-C_REVA
- removed L4: 0.47uH, robot:Vishay-IHLP-2020BZ-FP_1.905x2.79-3D_2.0-0-0-MFG, symbol robot:INDUCTOR
- removed NT5 (x2): NetTie_2, robot:NetTie-_SMD_Pad6mil, symbol Device:NetTie_2
- removed R12: 100k, robot:R_0603_1608Metric, symbol robot:R
- removed R13: DNP, robot:R_0603_1608Metric, symbol robot:R
- removed R32, R33: 10, robot:R_0402_1005Metric, symbol robot:R
- removed R34, R35: 2.2k, robot:R_0603_1608Metric, symbol robot:R
- removed R36: 200k, robot:R_0603_1608Metric, symbol robot:R
- removed R37, R39: 649k, robot:R_0603_1608Metric, symbol robot:R
- removed R38, R40: 120k, robot:R_0603_1608Metric, symbol robot:R
- removed R65: 10M, robot:R_0603_1608Metric, symbol robot:R
- removed R73 (x2): 0, robot:R_0805_2012Metric, symbol Device:R
- removed R89 (x2): 0, robot:R_0603_1608Metric, symbol Device:R
- removed R95: 0, robot:R_0603_1608Metric_3pin_Switch, symbol robot:Switch_R_SMD_3pin
- removed S4: JS202011JCQN, robot:SW_JS202011JCQN, symbol robot:JS202011SCQN
- removed TP13, TP14, TP15, TP3, TP4, TP5, TP6, TP7, TP8: SMD_0603, robot:TestPoint_SMD_0603, symbol robot:TestPoint
- removed U11: MAX77958EWV+T, robot:MAX77958EWV&plus_T, symbol robot:MAX77958EWV+T
- removed U15, U20: TPD1E05U06, robot:TPD1E05U06DPYR, symbol robot:TPD1E05U06
- removed U16: fpf1048bucx, robot:BGA6N50P3X2_146X96X62N, symbol robot:fpf1048bucx
- removed U17: TPS61253AYFFT, robot:Texas_Instruments-YFF0009-BGA9C40P3X3_119X129X62, symbol robot:TPS61253AYFFR
- removed U19, U21, U22, U23: TPD1E05U06, robot:TPD1E05U06DPYR, symbol robot:TPD1E05U06_1
- removed U24: TVS0500DRV, robot:TVS0500DRVR, symbol robot:TVS0500DRV
- added J9: Conn_01x16, robot:SMD FOR CASTELLATED 1x16 2.54mm, symbol Connector_Generic:Conn_01x16
Connections:
- net AGND: now also J9.10 (Pin_10)
- net DN1: now also J9.16 (Pin_16)
- net DP1: now also J9.15 (Pin_15)
- net INTB_SL: now also J9.9 (Pin_9)
- net SCL_M: now also J9.7 (Pin_7)
- net SCL_SL: now also J9.13 (Pin_13)
- net SDA_M: now also J9.8 (Pin_8)
- net SDA_SL: now also J9.14 (Pin_14)
- net USB_Phone_SYS: now also J9.1 (Pin_1), J9.2 (Pin_2)
- net VCIN: now also J9.6 (Pin_6)
- net VIO1: now also J9.12 (Pin_12)
- net VIO2: now also J9.11 (Pin_11)
- new net PGND: J9.3 (Pin_3), J9.4 (Pin_4)
- no-connect marks 11 -> 0
Other:
- note added: "AGND"
- note added: "DN1"
- note added: "DP1"
- note added: "INTB_SL"
- note added: "PGND"
- note added: "SCL_M"
- note added: "SCL_SL"
- note added: "SDA_M"
- note added: "SDA_SL"
- note added: "This is the connector for the new external USB PD Phone module."
- note added: "USB_Phone_SYS"
- note added: "VCIN"
- note added: "VIO1"
- note added: "VIO2"
- note removed: "Enable takes 500 us or so. For FRS you need to be less than 150 So GPIO0 needs to be on prior to the FRS request is sent."
- note removed: "Looks like VIN_5V pulls up to 16 mA to program the MTP whereas all other power comes from SYS or VBUS with VBUS taking precedence"
- note removed: "Move both jumpers to toggle between directly connecting USB port D+/- with MCU vs gated."
- note removed: "Pull ups based on single slave device and reducing power consumption."
- note removed: "This should be kept low else back currents can occur Only test Forced PWM or Ultrasonic if you ensure no source present on VOUT"
