File: pcb/robot/USB-PD-PhonePC.kicad_sch (KiCad schematic)
At the start: 1 part, among them J9 Conn_01x16

Commit message: Project and document update
Parts:
- J9: now left out of the parts list
Connections:
- no-connect marks 0 -> 1
Changed lines of the file:
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@@
 		(color 0 0 0 0)
+	)
+	(no_connect
+		(at 293.37 195.58)
 	)
 	(wire
@@
 		(unit 1)
 		(exclude_from_sim no)
-		(in_bom yes)
+		(in_bom no)
 		(on_board yes)
 		(dnp no)
