File: pcb/robot/boostRegulator.kicad_sch (KiCad schematic)
At the start: 21 parts, among them U5 LSF0102DCTR, U6 MAX77857BEWB+

Commit message: Modularized usb-pd board and main board split
Parts:
- renumbered C74 to C91, NT5 to NT15, TP18 to TP19
