File: pcb/robot/boostRegulator.kicad_sch (KiCad schematic)
At the start: 21 parts, among them U5 LSF0102DCTR, U6 MAX77857BEWB+

Commit message: Add removable I2C isolation jumpers on i2c0 and i2c1 (fixes #18)
Add a 0-ohm series resistor on both SDA and SCL for each slave on the
shared I2C buses, so a specific device can be isolated during
debugging (bus lockup / SDA-held-low) by pulling one resistor instead
of physical rework.

i2c0: R32/R33 (U1, STWLC38), R34/R35 (U12, fuel gauge), R36/R37 (U8,
motor driver), R38/R39 (U9, motor driver), R40/R53 (U6, MAX77857 -
placed between the level-shifter U5 and U6 so it isolates only that
branch). J9's existing link to the USB-PD module (R6/R7) was already
covered, no new jumper needed there.

i2c1: R55/R57 (U13, MAX77976 charger) and R65/R73 (J9's other I2C
link to the USB-PD module) - extended to this bus too, not just
i2c0 as the issue literally named, since the same lockup risk applies.

All 10 are 0-ohm, 0603, populated by default - only pull the one for
the suspect device during debugging. Placed for hand accessibility
where board space allowed.

Verified via ERC/DRC against the pre-#18 baseline: 0 unconnected
items, no new violations (318 ERC / 27 DRC, unchanged).

Co-Authored-By: Claude Sonnet 5 <noreply@anthropic.com>
Parts:
- added R40, R53: 0, robot:R_0603_1608Metric, symbol Device:R
Connections:
- net at R21.2, U6.A1 (SCL): now also R53.2; no longer TP18.1, U5.3 (A1)
- net at R20.2, U6.B1 (SDA): now also R40.2; no longer TP19.1, U5.4 (A2)
- new net: R53.1, TP18.1, U5.3 (A1)
- new net: R40.1, TP19.1, U5.4 (A2)
Changed lines of the file:
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@@
 	(text "Don't need.\nCan read everything we need from I2C"
 		(exclude_from_sim no)
-		(at 133.35 127 0)
+		(at 127.254 126.746 0)
 		(effects
 			(font
@@
 	)
 	(junction
-		(at 97.79 129.54)
+		(at 153.035 90.17)
 		(diameter 0)
 		(color 0 0 0 0)
 	)
 	(junction
-		(at 153.035 90.17)
+		(at 97.79 129.54)
 		(diameter 0)
 		(color 0 0 0 0)
@@
 	)
 	(junction
+		(at 97.79 127)
+		(diameter 0)
+		(color 0 0 0 0)
+	)
+	(junction
+		(at 121.285 127)
+		(diameter 0)
+		(color 0 0 0 0)
+	)
+	(junction
 		(at 191.77 140.97)
 		(diameter 0)
@@
 	)
 	(junction
+		(at 112.395 129.54)
+		(diameter 0)
+		(color 0 0 0 0)
+	)
+	(junction
 		(at 266.7 90.17)
 		(diameter 0)
@@
 	)
 	(junction
-		(at 97.79 127)
-		(diameter 0)
-		(color 0 0 0 0)
-	)
-	(junction
 		(at 125.095 90.17)
 		(diameter 0)
@@
 	)
 	(junction
-		(at 121.285 127)
-		(diameter 0)
-		(color 0 0 0 0)
-	)
-	(junction
 		(at 204.47 80.01)
 		(diameter 0)
@@
 	)
 	(junction
-		(at 112.395 129.54)
-		(diameter 0)
-		(color 0 0 0 0)
-	)
-	(junction
 		(at 171.45 95.25)
 		(diameter 0)
@@
 	(wire
 		(pts
-			(xy 112.395 129.54) (xy 171.45 129.54)
+			(xy 144.78 104.14) (xy 171.45 104.14)
 		)
 		(stroke
@@
 	(wire
 		(pts
-			(xy 144.78 104.14) (xy 171.45 104.14)
+			(xy 218.44 95.25) (xy 218.44 97.79)
 		)
 		(stroke
@@
 	(wire
 		(pts
-			(xy 218.44 95.25) (xy 218.44 97.79)
+			(xy 112.395 129.54) (xy 171.45 129.54)
 		)
 		(stroke
@@
 	(wire
 		(pts
-			(xy 97.79 129.54) (xy 112.395 129.54)
+			(xy 109.22 127) (xy 121.285 127)
 		)
 		(stroke
@@
 	(wire
 		(pts
-			(xy 97.79 127) (xy 121.285 127)
+			(xy 97.79 127) (xy 101.6 127)
+		)
+		(stroke
+			(width 0)
+			(type default)
+		)
+	)
+	(wire
+		(pts
+			(xy 109.22 129.54) (xy 112.395 129.54)
+		)
+		(stroke
+			(width 0)
+			(type default)
+		)
+	)
+	(wire
+		(pts
+			(xy 97.79 129.54) (xy 101.6 129.54)
 		)
 		(stroke
@@
 	)
 	(symbol
+		(lib_id "Device:R")
+		(at 105.41 129.54 90)
+		(unit 1)
+		(exclude_from_sim no)
+		(in_bom yes)
+		(on_board yes)
+		(dnp no)
+		(property "Reference" "R40"
+			(at 105.664 131.826 90)
+			(effects
+				(font
+					(size 1.27 1.27)
+				)
+			)
+		)
+		(property "Value" "0"
+			(at 105.41 129.54 90)
+			(effects
+				(font
+					(size 1.27 1.27)
+				)
+			)
+		)
+		(property "Footprint" "robot:R_0603_1608Metric"
+			(at 105.41 131.318 90)
+			(effects
+				(font
+					(size 1.27 1.27)
+				)
+				(hide yes)
+			)
+		)
+		(property "Datasheet" "~"
+			(at 105.41 129.54 0)
+			(effects
+				(font
+					(size 1.27 1.27)
+				)
+				(hide yes)
+			)
+		)
+		(property "Description" ""
+			(at 105.41 129.54 0)
+			(effects
+				(font
+					(size 1.27 1.27)
+				)
+			)
+		)
+		(property "Manufacturer" "Stackpole Electronics"
+			(at 105.41 129.54 90)
+			(effects
+				(font
+					(size 1.27 1.27)
+				)
+				(hide yes)
+			)
+		)
+		(property "Part Number" "RMCF0603ZT0R00"
+			(at 105.41 129.54 90)
+			(effects
+				(font
+					(size 1.27 1.27)
+				)
+				(hide yes)
+			)
+		)
+		(property "Stock" "15"
+			(at 105.41 129.54 0)
+			(effects
+				(font
+					(size 1.27 1.27)
+				)
+				(hide yes)
+			)
+		)
+		(property "Type" "SMD"
+			(at 105.41 129.54 0)
+			(effects
+				(font
+					(size 1.27 1.27)
+				)
+				(hide yes)
+			)
+		)
+		(pin "1"
+		)
+		(pin "2"
+		)
+		(instances
+			(project "robot"
+				(path "/0c7b298e-2d07-4b1f-b033-e95f02d45089/427922e5-a943-4728-8788-709c0c3b2395"
+					(reference "R40")
+					(unit 1)
+				)
+			)
+		)
+	)
+	(symbol
 		(lib_id "robot:R")
 		(at 112.395 115.57 0)
@@
 		(dnp no)
 		(property "Reference" "TP19"
-			(at 100.33 134.112 0)
+			(at 98.552 134.112 0)
 			(effects
 				(font
 					(size 1.27 1.27)
 				)
-				(justify left)
+				(justify right)
 			)
 		)
 		(property "Value" "SMD_0603"
-			(at 100.33 131.572 0)
+			(at 94.742 135.89 0)
 			(effects
 				(font
@@
 		(on_board yes)
 		(dnp no)
-		(fields_autoplaced yes)
 		(property "Reference" "TP18"
 			(at 100.33 122.428 0)
@@
 		)
 		(property "Value" "SMD_0603"
-			(at 100.33 124.968 0)
+			(at 92.71 120.904 0)
 			(effects
 				(font
@@
 					(unit 1)
 				)
+			)
+		)
+	)
+	(symbol
+		(lib_id "Device:R")
+		(at 105.41 127 90)
+		(unit 1)
+		(exclude_from_sim no)
+		(in_bom yes)
+		(on_board yes)
+		(dnp no)
+		(property "Reference" "R53"
+			(at 105.41 124.46 90)
+			(effects
+				(font
+					(size 1.27 1.27)
+				)
+			)
+		)
+		(property "Value" "0"
+			(at 105.41 127 90)
+			(effects
+				(font
+					(size 1.27 1.27)
+				)
+			)
+		)
+		(property "Footprint" "robot:R_0603_1608Metric"
+			(at 105.41 128.778 90)
+			(effects
+				(font
+					(size 1.27 1.27)
+				)
+				(hide yes)
+			)
+		)
+		(property "Datasheet" "~"
+			(at 105.41 127 0)
+			(effects
+				(font
+					(size 1.27 1.27)
+				)
+				(hide yes)
+			)
+		)
+		(property "Description" ""
+			(at 105.41 127 0)
+			(effects
+				(font
+					(size 1.27 1.27)
+				)
+			)
+		)
+		(property "Manufacturer" "Stackpole Electronics"
+			(at 105.41 127 90)
+			(effects
+				(font
+					(size 1.27 1.27)
+				)
+				(hide yes)
+			)
+		)
+		(property "Part Number" "RMCF0603ZT0R00"
+			(at 105.41 127 90)
+			(effects
+				(font
+					(size 1.27 1.27)
+				)
+				(hide yes)
+			)
+		)
+		(property "Stock" "15"
+			(at 105.41 127 0)
+			(effects
+				(font
+					(size 1.27 1.27)
+				)
+				(hide yes)
+			)
+		)
+		(property "Type" "SMD"
+			(at 105.41 127 0)
+			(effects
+				(font
+					(size 1.27 1.27)
+				)
+				(hide yes)
+			)
+		)
+		(pin "1"
+		)
+		(pin "2"
+		)
+		(instances
+			(project "robot"
+				(path "/0c7b298e-2d07-4b1f-b033-e95f02d45089/427922e5-a943-4728-8788-709c0c3b2395"
+					(reference "R53")
+					(unit 1)
+				)
