File: pcb/robot/robot.kicad_sch (KiCad schematic)
At the start: 53 parts, among them U7 AP2502KTR-G1

Commit message: Modularized usb-pd board and main board split
Parts:
- renumbered NT5 to NT14, NT5 to NT16, NT5 to NT18, NT5 to NT20, TP16 to TP1, TP16 to TP17, TP16 to TP2, TP18 to TP20, TP18 to TP21, TP23 to TP30, TP23 to TP34, TP23 to TP39, TP23 to TP40, TP23 to TP41, TP23 to TP42, TP23 to TP43
Other:
- note added: "This is an external module."
