File: pcb/robot/robot.kicad_sch (KiCad schematic)
At the start: 53 parts, among them U7 AP2502KTR-G1

Commit message: Replace ADC charger-sense front-end with GPIO interrupts (fixes #19)
Add 2x TPS3808G01DBVR voltage supervisors on USB_V and VRect
charger-sense paths, replacing the ADC divider+RC filter. GPIO26_ADC0/
GPIO27_ADC1 are now digital interrupt inputs (VIT~4.46V USB_V,
~2.11V VRect) instead of ADC channels.

Renamed net labels to reflect the digital nature of these signals:
ADC0 -> USB_SNS, ADC1 -> WLC_SNS (both hierarchical, crossing into
the MCU sheet), GPIO26_ADC0 -> GPIO26_USB_INT, GPIO27_ADC1 ->
GPIO27_WLC_INT (local labels). Documented the new circuit, threshold
derivation, and firmware implications in a schematic note replacing
the old #14-era one.

Verified via ERC/DRC against the pre-#19 baseline: 0 unconnected
items, no new error-level violations - only cosmetic silkscreen
warnings from the imported LCSC footprints.

Co-Authored-By: Claude Sonnet 5 <noreply@anthropic.com>
Other:
- sheet MCU ports: added USB_SNS, WLC_SNS; removed ADC0, ADC1
Changed lines of the file:
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@@
 		)
 	)
-	(label "ADC0"
+	(label "USB_SNS"
 		(at 127 46.99 180)
 		(effects
@@
 		)
 	)
-	(label "ADC0"
+	(label "USB_SNS"
 		(at 182.88 111.76 180)
 		(effects
@@
 			)
 		)
-		(pin "ADC0" input
+		(pin "USB_SNS" input
 			(at 172.72 111.76 0)
 			(effects
@@
 			)
 		)
-		(pin "ADC1" input
+		(pin "WLC_SNS" input
 			(at 148.59 127 180)
 			(effects
