File: pcb/robot/robot.kicad_sch (KiCad schematic)
At the start: 53 parts, among them U7 AP2502KTR-G1

Commit message: Re-unify USB-PD module into main board (single-PCB architecture) (#17)
Merges the USB-PD module circuitry back into the main robot board as
a single PCB, reversing the earlier main-board/USB-PD-daughter-board
split. Full re-route and re-placement of the combined design:

- Consolidated low-profile parts toward the board center, using the
  space freed up by relocated capacitors, for better overall use of
  the available area.
- Kept all 0-ohm test/isolation jumpers in accessible locations for
  bench testing.
- Added/corrected footprints for several parts that had broken or
  incorrect footprints (DDC6_TEX variants, SOT-23-6, SOT-23-3,
  R0402).

Carries forward every closed correction issue and update made since
the original split: #3 (CC jumpers), #6 (IC1.ON pull-down), #14/#15
(ADC divider, motor connector pinout), #16, #18 (I2C isolation
jumpers), #19 (charger-sense GPIO interrupt), plus the BOM/pricing
updates, LED changes, and MAX77642 replacement.

Verified via kicad-cli ERC/DRC + netlist diff against the pre-merge
board: 0 unconnected items (unchanged), no new DRC error-level
violations besides one pre-existing excluded item, and the #6
(IC1.ON pull-down) and #19 (charger-sense GPIO interrupt) circuits
confirmed intact at the net-topology level despite the full-board
re-annotation changing most reference designators. Most of the raw
diff size is a KiCad 9 footprint-format upgrade (pre-2023 format
rewritten to current) rather than design changes - spot-checked
against unrelated footprints (e.g. mounting holes), which show
identical geometry under the new syntax.
Parts:
- NT1: renamed from NT20; symbol Device:NetTie_2 -> robot:NetTie_2
- NT2: renamed from NT18; symbol Device:NetTie_2 -> robot:NetTie_2
- NT3: renamed from NT14; symbol Device:NetTie_2 -> robot:NetTie_2
- NT4: renamed from NT16; symbol Device:NetTie_2 -> robot:NetTie_2
- R1: renamed from R52; symbol Device:R -> robot:R
- R10: renamed from R78; symbol Device:R -> robot:R
- R11: renamed from R76; symbol Device:R -> robot:R
- R12: renamed from R67; symbol Device:R -> robot:R
- R13: renamed from R68; symbol Device:R -> robot:R
- R14: renamed from R86; symbol Device:R -> robot:R
- R15: renamed from R79; symbol Device:R -> robot:R
- R16: renamed from R80; symbol Device:R -> robot:R
- R17: renamed from R81; symbol Device:R -> robot:R
- R18: renamed from R88; symbol Device:R -> robot:R
- R19: renamed from R11; symbol Device:R -> robot:R
- R2: renamed from R54; symbol Device:R -> robot:R
- R20: renamed from R69; symbol Device:R -> robot:R
- R21: renamed from R70; symbol Device:R -> robot:R
- R22: renamed from R82; symbol Device:R -> robot:R
- R23: renamed from R83; symbol Device:R -> robot:R
- R24: renamed from R71; symbol Device:R -> robot:R
- R25: renamed from R72; symbol Device:R -> robot:R
- R26: renamed from R84; symbol Device:R -> robot:R
- R27: renamed from R85; symbol Device:R -> robot:R
- R5: renamed from R90; symbol Device:R -> robot:R
- R8: renamed from R87; symbol Device:R -> robot:R
- R9: renamed from R77; symbol Device:R -> robot:R
- renumbered R6 to R3, R7 to R4, R14 to R6, R15 to R7, S3 to S1, TP39 to TP1, TP41 to TP10, TP42 to TP11, TP43 to TP12, TP34 to TP13, TP40 to TP2, TP16 to TP3, TP1 to TP4, TP20 to TP5, TP21 to TP6, TP2 to TP7, TP17 to TP8, TP30 to TP9, U7 to U1

Commit message: Add switch-open discharge detector and low-power OV reference (#22, #23)
U34 (new, MCP6541 on IC1-VBIAS) senses the power switch via
Net-(IC1-ON) and forces Q7/R124 (#22's shunt) to discharge
/MOTORS/VCC when the switch opens, independent of the 3V3 rail.
OR'd into Q7's gate through D11/D12 alongside U32's existing
overvoltage trip - discharges in ~2.2ms vs. the ~500-600ms the
MAX77857 was timing out at.

Also swaps U33 (TLVH431) for a MAX6006A micropower reference and
bumps R131 to 412k, per Christopher's request on #22 - cuts the
clamp's standing current from ~218uA to ~18uA with the same
5.6V/5.4V thresholds.

Verified with kicad-cli: ERC clean, 0 unconnected items, schematic
parity clean (pre-existing U12 footprint mismatch aside).
Other:
- sheet MOTORS ports: added SHDN; removed none
- sheet Protection ports: added SHDN; removed none
Changed lines of the file:
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@@
 		)
 	)
+	(wire
+		(pts
+			(xy 220.98 99.06) (xy 229.87 99.06)
+		)
+		(stroke
+			(width 0)
+			(type default)
+		)
+	)
 	(bus
 		(pts
@@
 	(wire
 		(pts
+			(xy 72.39 67.31) (xy 78.74 67.31)
+		)
+		(stroke
+			(width 0)
+			(type default)
+		)
+	)
+	(wire
+		(pts
 			(xy 213.36 125.73) (xy 212.09 125.73)
 		)
@@
 		)
 	)
+	(label "SHDN"
+		(at 72.39 67.31 0)
+		(effects
+			(font
+				(size 1.27 1.27)
+			)
+			(justify left bottom)
+		)
+	)
 	(label "AGND"
 		(at 110.49 191.135 0)
@@
 		)
 	)
+	(label "SHDN"
+		(at 220.98 99.06 0)
+		(effects
+			(font
+				(size 1.27 1.27)
+			)
+			(justify left bottom)
+		)
+	)
 	(label "I2C0_SCL"
 		(at 219.71 55.88 0)
@@
 			)
 		)
+		(pin "SHDN" input
+			(at 229.87 99.06 180)
+			(effects
+				(font
+					(size 1.27 1.27)
+				)
+				(justify left)
+			)
+		)
 		(instances
 			(project "robot"
@@
 			)
 		)
+		(pin "SHDN" input
+			(at 78.74 67.31 180)
+			(effects
+				(font
+					(size 1.27 1.27)
+				)
+				(justify left)
+			)
+		)

Commit message: Gate MAX77857 EN via GPIO22 divider, bump C136 to 100nF (#24)
R135/R136 (10k/10k) now gate U23.EN from GPIO22 instead of tying it
straight to 1.8V. GPIO22 low or floating (RP2040 reset/boot default)
holds EN at 0V, no firmware dependency for the off-state. VIO stays
on 1.8V, untouched. C136 220pF -> 100nF (CL05A104KA5NNNC) to meet
the MAX6006's real >=10nF minimum.

Verified against baseline: ERC 337/337 (no new violations), DRC 0
unconnected items, no violations tied to the new parts.
Other:
- sheet BoostRegulator ports: added GPIO22; removed none
- sheet MCU ports: added GPIO22; removed none
Changed lines of the file:
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@@
 	(wire
 		(pts
+			(xy 220.98 50.8) (xy 229.87 50.8)
+		)
+		(stroke
+			(width 0)
+			(type default)
+		)
+	)
+	(wire
+		(pts
 			(xy 139.7 119.38) (xy 148.59 119.38)
 		)
@@
 	(wire
 		(pts
+			(xy 172.72 115.57) (xy 176.53 115.57)
+		)
+		(stroke
+			(width 0)
+			(type default)
+		)
+	)
+	(wire
+		(pts
 			(xy 107.315 99.06) (xy 107.315 93.98)
 		)
@@
 		)
 	)
-	(wire
-		(pts
-			(xy 139.7 127) (xy 148.59 127)
-		)
-		(stroke
-			(width 0)
-			(type default)
-		)
-	)
 	(bus
 		(pts
@@
 	(wire
 		(pts
-			(xy 139.7 129.54) (xy 148.59 129.54)
-		)
-		(stroke
-			(width 0)
-			(type default)
-		)
-	)
-	(wire
-		(pts
 			(xy 116.205 123.19) (xy 124.46 123.19)
 		)
@@
 	(wire
 		(pts
+			(xy 139.7 129.54) (xy 148.59 129.54)
+		)
+		(stroke
+			(width 0)
+			(type default)
+		)
+	)
+	(wire
+		(pts
 			(xy 170.815 144.78) (xy 170.815 146.05)
 		)
@@
 	(wire
 		(pts
+			(xy 139.7 127) (xy 148.59 127)
+		)
+		(stroke
+			(width 0)
+			(type default)
+		)
+	)
+	(wire
+		(pts
 			(xy 116.205 99.06) (xy 116.205 93.98)
 		)
@@
 	)
 	(label "AGND"
-		(at 139.7 129.54 0)
+		(at 176.53 115.57 0)
 		(effects
 			(font
@@
 		)
 	)
+	(label "GPIO22"
+		(at 139.7 127 0)
+		(effects
+			(font
+				(size 1.27 1.27)
+			)
+			(justify left bottom)
+		)
+	)
 	(label "I2C0_SCL"
 		(at 219.71 55.88 0)
@@
 	)
 	(label "VRect"
-		(at 139.7 127 0)
+		(at 139.7 129.54 0)
 		(effects
 			(font
@@
 		)
 	)
+	(label "GPIO22"
+		(at 220.98 50.8 0)
+		(effects
+			(font
+				(size 1.27 1.27)
+			)
+			(justify left bottom)
+		)
+	)
 	(label "GPIO20"
 		(at 139.7 119.38 0)
@@
 			)
 		)
+		(pin "GPIO22" input
+			(at 229.87 50.8 180)
+			(effects
+				(font
+					(size 1.27 1.27)
+				)
+				(justify left)
+			)
+		)
 		(instances
 			(project "robot"
@@
 		)
 		(pin "GND" input
-			(at 148.59 129.54 180)
+			(at 172.72 115.57 0)
 			(effects
 				(font
 					(size 1.27 1.27)
 				)
-				(justify left)
+				(justify right)
 			)
 		)
@@
 		)
 		(pin "WLC_SNS" input
+			(at 148.59 129.54 180)
+			(effects
+				(font
+					(size 1.27 1.27)
+				)
+				(justify left)
+			)
+		)
+		(pin "GPIO22" input
 			(at 148.59 127 180)
 			(effects
