File: pcb/robot/powerMux.kicad_sch (KiCad schematic)
At the start: 8 parts, among them Q1 Q_NMOS_GDS, U4 NCP3901

Commit message: Replace ADC charger-sense front-end with GPIO interrupts (fixes #19)
Add 2x TPS3808G01DBVR voltage supervisors on USB_V and VRect
charger-sense paths, replacing the ADC divider+RC filter. GPIO26_ADC0/
GPIO27_ADC1 are now digital interrupt inputs (VIT~4.46V USB_V,
~2.11V VRect) instead of ADC channels.

Renamed net labels to reflect the digital nature of these signals:
ADC0 -> USB_SNS, ADC1 -> WLC_SNS (both hierarchical, crossing into
the MCU sheet), GPIO26_ADC0 -> GPIO26_USB_INT, GPIO27_ADC1 ->
GPIO27_WLC_INT (local labels). Documented the new circuit, threshold
derivation, and firmware implications in a schematic note replacing
the old #14-era one.

Verified via ERC/DRC against the pre-#19 baseline: 0 unconnected
items, no new error-level violations - only cosmetic silkscreen
warnings from the imported LCSC footprints.

Co-Authored-By: Claude Sonnet 5 <noreply@anthropic.com>
Parts:
- R16: value 510k -> 1M; Part Number RMCF0603JT510K -> FRC0603F1004TS
Changed lines of the file:
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@@
 			)
 		)
-		(property "Value" "510k"
+		(property "Value" "1M"
 			(at 176.53 124.4599 0)
 			(effects
@@
 			)
 		)
-		(property "Part Number" "RMCF0603JT510K"
+		(property "Part Number" "FRC0603F1004TS"
 			(at 173.99 123.19 0)
 			(effects
