File: pcb/robot/powerMux.kicad_sch (KiCad schematic)
At the start: 8 parts, among them Q1 Q_NMOS_GDS, U4 NCP3901

Commit message: Re-unify USB-PD module into main board (single-PCB architecture) (#17)
Merges the USB-PD module circuitry back into the main robot board as
a single PCB, reversing the earlier main-board/USB-PD-daughter-board
split. Full re-route and re-placement of the combined design:

- Consolidated low-profile parts toward the board center, using the
  space freed up by relocated capacitors, for better overall use of
  the available area.
- Kept all 0-ohm test/isolation jumpers in accessible locations for
  bench testing.
- Added/corrected footprints for several parts that had broken or
  incorrect footprints (DDC6_TEX variants, SOT-23-6, SOT-23-3,
  R0402).

Carries forward every closed correction issue and update made since
the original split: #3 (CC jumpers), #6 (IC1.ON pull-down), #14/#15
(ADC divider, motor connector pinout), #16, #18 (I2C isolation
jumpers), #19 (charger-sense GPIO interrupt), plus the BOM/pricing
updates, LED changes, and MAX77642 replacement.

Verified via kicad-cli ERC/DRC + netlist diff against the pre-merge
board: 0 unconnected items (unchanged), no new DRC error-level
violations besides one pre-existing excluded item, and the #6
(IC1.ON pull-down) and #19 (charger-sense GPIO interrupt) circuits
confirmed intact at the net-topology level despite the full-board
re-annotation changing most reference designators. Most of the raw
diff size is a KiCad 9 footprint-format upgrade (pre-2023 format
rewritten to current) rather than design changes - spot-checked
against unrelated footprints (e.g. mounting holes), which show
identical geometry under the new syntax.
Parts:
- renumbered C21 to C23, C22 to C24, C23 to C25, R16 to R53, R17 to R54, R18 to R55, U4 to U14
Changed lines of the file:
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@@
 		(dnp no)
 		(fields_autoplaced yes)
-		(property "Reference" "R16"
+		(property "Reference" "R53"
 			(at 176.53 121.9199 0)
 			(effects
@@
 			(project "robot"
 				(path "/0c7b298e-2d07-4b1f-b033-e95f02d45089/e17fda7c-211f-4188-9d42-b948f78009dd"
-					(reference "R16")
+					(reference "R53")
 					(unit 1)
 				)
@@
 		(on_board yes)
 		(dnp no)
-		(property "Reference" "C23"
+		(property "Reference" "C25"
 			(at 170.18 92.7099 0)
 			(effects
@@
 			(project "robot"
 				(path "/0c7b298e-2d07-4b1f-b033-e95f02d45089/e17fda7c-211f-4188-9d42-b948f78009dd"
-					(reference "C23")
+					(reference "C25")
 					(unit 1)
 				)
@@
 		(on_board yes)
 		(dnp no)
-		(property "Reference" "C22"
+		(property "Reference" "C24"
 			(at 115.57 113.0299 0)
 			(effects
@@
 			(project "robot"
 				(path "/0c7b298e-2d07-4b1f-b033-e95f02d45089/e17fda7c-211f-4188-9d42-b948f78009dd"
-					(reference "C22")
+					(reference "C24")
 					(unit 1)
 				)
@@
 		(dnp no)
 		(fields_autoplaced yes)
-		(property "Reference" "R18"
+		(property "Reference" "R55"
 			(at 212.09 66.0399 0)
 			(effects
@@
 			(project "robot"
 				(path "/0c7b298e-2d07-4b1f-b033-e95f02d45089/e17fda7c-211f-4188-9d42-b948f78009dd"
-					(reference "R18")
+					(reference "R55")
 					(unit 1)
 				)
@@
 		(on_board yes)
 		(dnp no)
-		(property "Reference" "C21"
+		(property "Reference" "C23"
 			(at 80.01 96.5199 0)
 			(effects
@@
 			(project "robot"
 				(path "/0c7b298e-2d07-4b1f-b033-e95f02d45089/e17fda7c-211f-4188-9d42-b948f78009dd"
-					(reference "C21")
+					(reference "C23")
 					(unit 1)
 				)
@@
 		(dnp no)
 		(fields_autoplaced yes)
-		(property "Reference" "U4"
+		(property "Reference" "U14"
 			(at 140.335 73.66 0)
 			(effects
@@
 			(project "robot"
 				(path "/0c7b298e-2d07-4b1f-b033-e95f02d45089/e17fda7c-211f-4188-9d42-b948f78009dd"
-					(reference "U4")
+					(reference "U14")
 					(unit 1)
 				)
@@
 		(dnp no)
 		(fields_autoplaced yes)
-		(property "Reference" "R17"
+		(property "Reference" "R54"
 			(at 176.53 134.6199 0)
 			(effects
@@
 			(project "robot"
 				(path "/0c7b298e-2d07-4b1f-b033-e95f02d45089/e17fda7c-211f-4188-9d42-b948f78009dd"
-					(reference "R17")
+					(reference "R54")
 					(unit 1)
 				)
