File: pcb/robot/Wireless-Receiver.kicad_sch (KiCad schematic)
At the start: 49 parts, among them J8 Conn_01x02, U1 STWLC38JRM

Commit message: Add removable I2C isolation jumpers on i2c0 and i2c1 (fixes #18)
Add a 0-ohm series resistor on both SDA and SCL for each slave on the
shared I2C buses, so a specific device can be isolated during
debugging (bus lockup / SDA-held-low) by pulling one resistor instead
of physical rework.

i2c0: R32/R33 (U1, STWLC38), R34/R35 (U12, fuel gauge), R36/R37 (U8,
motor driver), R38/R39 (U9, motor driver), R40/R53 (U6, MAX77857 -
placed between the level-shifter U5 and U6 so it isolates only that
branch). J9's existing link to the USB-PD module (R6/R7) was already
covered, no new jumper needed there.

i2c1: R55/R57 (U13, MAX77976 charger) and R65/R73 (J9's other I2C
link to the USB-PD module) - extended to this bus too, not just
i2c0 as the issue literally named, since the same lockup risk applies.

All 10 are 0-ohm, 0603, populated by default - only pull the one for
the suspect device during debugging. Placed for hand accessibility
where board space allowed.

Verified via ERC/DRC against the pre-#18 baseline: 0 unconnected
items, no new violations (318 ERC / 27 DRC, unchanged).

Co-Authored-By: Claude Sonnet 5 <noreply@anthropic.com>
Parts:
- added R32, R33: 0, robot:R_0603_1608Metric, symbol Device:R
Connections:
- net SCL: now also R33.2; no longer U1.H5 (SCL)
- net SDA: now also R32.2; no longer U1.G5 (SDA)
- new net: R32.1, U1.G5 (SDA)
- new net: R33.1, U1.H5 (SCL)
Changed lines of the file:
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@@
 	(wire
 		(pts
+			(xy 147.32 163.83) (xy 149.86 163.83)
+		)
+		(stroke
+			(width 0)
+			(type default)
+		)
+	)
+	(wire
+		(pts
 			(xy 78.74 33.02) (xy 91.44 33.02)
 		)
@@
 	(wire
 		(pts
-			(xy 147.32 160.02) (xy 151.13 160.02)
-		)
-		(stroke
-			(width 0)
-			(type default)
-		)
-	)
-	(wire
-		(pts
 			(xy 36.83 44.45) (xy 36.83 46.99)
 		)
@@
 	(wire
 		(pts
+			(xy 147.32 160.02) (xy 149.86 160.02)
+		)
+		(stroke
+			(width 0)
+			(type default)
+		)
+	)
+	(wire
+		(pts
 			(xy 77.47 130.81) (xy 77.47 133.35)
 		)
@@
 	(wire
 		(pts
-			(xy 147.32 163.83) (xy 151.13 163.83)
+			(xy 165.1 124.46) (xy 175.26 124.46)
 		)
 		(stroke
@@
 	(wire
 		(pts
-			(xy 165.1 124.46) (xy 175.26 124.46)
+			(xy 102.87 81.28) (xy 102.87 82.55)
 		)
 		(stroke
@@
 	(wire
 		(pts
-			(xy 102.87 81.28) (xy 102.87 82.55)
+			(xy 157.48 163.83) (xy 160.02 163.83)
 		)
 		(stroke
@@
 	(wire
 		(pts
+			(xy 157.48 160.02) (xy 160.02 160.02)
+		)
+		(stroke
+			(width 0)
+			(type default)
+		)
+	)
+	(wire
+		(pts
 			(xy 187.96 121.92) (xy 187.96 125.73)
 		)
@@
 	(hierarchical_label "SDA"
 		(shape input)
-		(at 151.13 160.02 0)
+		(at 160.02 160.02 0)
 		(effects
 			(font
@@
 	(hierarchical_label "SCL"
 		(shape input)
-		(at 151.13 163.83 0)
+		(at 160.02 163.83 0)
 		(effects
 			(font
@@
 	)
 	(symbol
+		(lib_id "Device:R")
+		(at 153.67 163.83 90)
+		(unit 1)
+		(exclude_from_sim no)
+		(in_bom yes)
+		(on_board yes)
+		(dnp no)
+		(property "Reference" "R33"
+			(at 153.924 166.116 90)
+			(effects
+				(font
+					(size 1.27 1.27)
+				)
+			)
+		)
+		(property "Value" "0"
+			(at 153.67 163.83 90)
+			(effects
+				(font
+					(size 1.27 1.27)
+				)
+			)
+		)
+		(property "Footprint" "robot:R_0603_1608Metric"
+			(at 153.67 165.608 90)
+			(effects
+				(font
+					(size 1.27 1.27)
+				)
+				(hide yes)
+			)
+		)
+		(property "Datasheet" "~"
+			(at 153.67 163.83 0)
+			(effects
+				(font
+					(size 1.27 1.27)
+				)
+				(hide yes)
+			)
+		)
+		(property "Description" ""
+			(at 153.67 163.83 0)
+			(effects
+				(font
+					(size 1.27 1.27)
+				)
+			)
+		)
+		(property "Manufacturer" "Stackpole Electronics"
+			(at 153.67 163.83 90)
+			(effects
+				(font
+					(size 1.27 1.27)
+				)
+				(hide yes)
+			)
+		)
+		(property "Part Number" "RMCF0603ZT0R00"
+			(at 153.67 163.83 90)
+			(effects
+				(font
+					(size 1.27 1.27)
+				)
+				(hide yes)
+			)
+		)
+		(property "Stock" "15"
+			(at 153.67 163.83 0)
+			(effects
+				(font
+					(size 1.27 1.27)
+				)
+				(hide yes)
+			)
+		)
+		(property "Type" "SMD"
+			(at 153.67 163.83 0)
+			(effects
+				(font
+					(size 1.27 1.27)
+				)
+				(hide yes)
+			)
+		)
+		(pin "1"
+		)
+		(pin "2"
+		)
+		(instances
+			(project "robot"
+				(path "/0c7b298e-2d07-4b1f-b033-e95f02d45089/d5c9d5c0-7de4-474c-9ba2-6b466f104c70"
+					(reference "R33")
+					(unit 1)
+				)
+			)
+		)
+	)
+	(symbol
 		(lib_id "robot:C")
 		(at 215.9 120.65 0)
@@
 					(unit 1)
 				)
+			)
+		)
+	)
+	(symbol
+		(lib_id "Device:R")
+		(at 153.67 160.02 90)
+		(unit 1)
+		(exclude_from_sim no)
+		(in_bom yes)
+		(on_board yes)
+		(dnp no)
+		(property "Reference" "R32"
+			(at 153.67 157.48 90)
+			(effects
+				(font
+					(size 1.27 1.27)
+				)
+			)
+		)
+		(property "Value" "0"
+			(at 153.67 160.02 90)
+			(effects
+				(font
+					(size 1.27 1.27)
+				)
+			)
+		)
+		(property "Footprint" "robot:R_0603_1608Metric"
+			(at 153.67 161.798 90)
+			(effects
+				(font
+					(size 1.27 1.27)
+				)
+				(hide yes)
+			)
+		)
+		(property "Datasheet" "~"
+			(at 153.67 160.02 0)
+			(effects
+				(font
+					(size 1.27 1.27)
+				)
+				(hide yes)
+			)
+		)
+		(property "Description" ""
+			(at 153.67 160.02 0)
+			(effects
+				(font
+					(size 1.27 1.27)
+				)
+			)
+		)
+		(property "Manufacturer" "Stackpole Electronics"
+			(at 153.67 160.02 90)
+			(effects
+				(font
+					(size 1.27 1.27)
+				)
+				(hide yes)
+			)
+		)
+		(property "Part Number" "RMCF0603ZT0R00"
+			(at 153.67 160.02 90)
+			(effects
+				(font
+					(size 1.27 1.27)
+				)
+				(hide yes)
+			)
+		)
+		(property "Stock" "15"
+			(at 153.67 160.02 0)
+			(effects
+				(font
+					(size 1.27 1.27)
+				)
+				(hide yes)
+			)
+		)
+		(property "Type" "SMD"
+			(at 153.67 160.02 0)
+			(effects
+				(font
+					(size 1.27 1.27)
+				)
+				(hide yes)
+			)
+		)
+		(pin "1"
+		)
+		(pin "2"
+		)
+		(instances
+			(project "robot"
+				(path "/0c7b298e-2d07-4b1f-b033-e95f02d45089/d5c9d5c0-7de4-474c-9ba2-6b466f104c70"
+					(reference "R32")
+					(unit 1)
+				)
