File: pcb/robot/Wireless-Receiver.kicad_sch (KiCad schematic)
At the start: 51 parts, among them J8 Conn_01x02, U1 STWLC38JRM

Commit message: Re-unify USB-PD module into main board (single-PCB architecture) (#17)
Merges the USB-PD module circuitry back into the main robot board as
a single PCB, reversing the earlier main-board/USB-PD-daughter-board
split. Full re-route and re-placement of the combined design:

- Consolidated low-profile parts toward the board center, using the
  space freed up by relocated capacitors, for better overall use of
  the available area.
- Kept all 0-ohm test/isolation jumpers in accessible locations for
  bench testing.
- Added/corrected footprints for several parts that had broken or
  incorrect footprints (DDC6_TEX variants, SOT-23-6, SOT-23-3,
  R0402).

Carries forward every closed correction issue and update made since
the original split: #3 (CC jumpers), #6 (IC1.ON pull-down), #14/#15
(ADC divider, motor connector pinout), #16, #18 (I2C isolation
jumpers), #19 (charger-sense GPIO interrupt), plus the BOM/pricing
updates, LED changes, and MAX77642 replacement.

Verified via kicad-cli ERC/DRC + netlist diff against the pre-merge
board: 0 unconnected items (unchanged), no new DRC error-level
violations besides one pre-existing excluded item, and the #6
(IC1.ON pull-down) and #19 (charger-sense GPIO interrupt) circuits
confirmed intact at the net-topology level despite the full-board
re-annotation changing most reference designators. Most of the raw
diff size is a KiCad 9 footprint-format upgrade (pre-2023 format
rewritten to current) rather than design changes - spot-checked
against unrelated footprints (e.g. mounting holes), which show
identical geometry under the new syntax.
Parts:
- D10: symbol Device:D_Zener -> robot:D_Zener
- D4: renamed from D11; symbol Device:D -> robot:D
- D5: renamed from D9; symbol Device:D -> robot:D
- D8: renamed from D4; symbol Device:D_Zener -> robot:D_Zener
- D9: renamed from D6; symbol Device:D_Zener -> robot:D_Zener
- R108: renamed from R32; symbol Device:R -> robot:R
- R109: renamed from R33; symbol Device:R -> robot:R
- renumbered C131 to C103, C132 to C104, C133 to C106, C134 to C109, C135 to C110, C136 to C114, C137 to C118, C138 to C121, C110 to C62, C111 to C63, C112 to C64, C109 to C69, C113 to C70, C114 to C72, C115 to C73, C116 to C76, C117 to C78, C118 to C79, C119 to C80, C120 to C81, C121 to C84, C122 to C85, C123 to C88, C124 to C91, C125 to C92, C126 to C93, C127 to C94, C128 to C95, C129 to C98, C130 to C99, J8 to J4, L5 to L4, R89 to R110, R103 to R111, R104 to R112, R105 to R113, R96 to R83, R98 to R84, R99 to R85, R100 to R86, R101 to R87, R102 to R89, U1 to U27
