File: pcb/robot/motors.kicad_sch (KiCad schematic)
At the start: 23 parts, among them J3 Conn_01x06_MountingPin, J5 Conn_01x06_MountingPin, J6 MotorCable, J7 MotorCable, Q6 SN74AHC125RGYR, U8 DRV8830DRCR, U9 DRV8830DRCR

Commit message: Add removable I2C isolation jumpers on i2c0 and i2c1 (fixes #18)
Add a 0-ohm series resistor on both SDA and SCL for each slave on the
shared I2C buses, so a specific device can be isolated during
debugging (bus lockup / SDA-held-low) by pulling one resistor instead
of physical rework.

i2c0: R32/R33 (U1, STWLC38), R34/R35 (U12, fuel gauge), R36/R37 (U8,
motor driver), R38/R39 (U9, motor driver), R40/R53 (U6, MAX77857 -
placed between the level-shifter U5 and U6 so it isolates only that
branch). J9's existing link to the USB-PD module (R6/R7) was already
covered, no new jumper needed there.

i2c1: R55/R57 (U13, MAX77976 charger) and R65/R73 (J9's other I2C
link to the USB-PD module) - extended to this bus too, not just
i2c0 as the issue literally named, since the same lockup risk applies.

All 10 are 0-ohm, 0603, populated by default - only pull the one for
the suspect device during debugging. Placed for hand accessibility
where board space allowed.

Verified via ERC/DRC against the pre-#18 baseline: 0 unconnected
items, no new violations (318 ERC / 27 DRC, unchanged).

Co-Authored-By: Claude Sonnet 5 <noreply@anthropic.com>
Parts:
- added R36, R37, R38, R39: 0, robot:R_0603_1608Metric, symbol Device:R
Connections:
- net SCL: now also R36.1, R38.1; no longer U8.10 (SCL), U9.10 (SCL)
- net SDA: now also R37.1, R39.1; no longer U8.9 (SDA), U9.9 (SDA)
- new net: R38.2, U9.10 (SCL)
- new net: R39.2, U9.9 (SDA)
- new net: R36.2, U8.10 (SCL)
- new net: R37.2, U8.9 (SDA)
