File: pcb/robot/motors.kicad_sch (KiCad schematic)
At the start: 45 parts, among them J5 MotorCable, J6 Conn_01x06_MountingPin, J7 Conn_01x06_MountingPin, J8 MotorCable, Q6 SN74AHC125RGYR, Q7 AO3400A, U25 DRV8830DRCR, U26 DRV8830DRCR, U32 MCP6541T-I/OT, U33 MAX6006AEUR+T

Commit message: Add OUT bypass cap on U33, move #23 divider away from L1 (#24)
C136 (220pF NP0, 0402) added across U33's OUT to speed up its
turn-on settling to ~200us - well ahead of the ~300us before
MAX77857 starts ramping VCC, per both real datasheets. EN stays
tied to 1V8, no gating circuit needed.

Also relocated U34/R125/R133 away from L1 (switching inductor,
different rail) - were under 1mm apart, now ~21mm.

Verified via kicad-cli: ERC unchanged (333/333), DRC 0 unconnected,
same pre-existing U12 parity warning only, no new electrical issues.
Parts:
- added C136: 220pF, easyeda2kicad:C0402, symbol easyeda2kicad:CC0402FRNPO9BN221
Connections:
- net PGND: now also C136.2
- net at R131.1, U32.4 (VIN-), U33.1 (OUT): now also C136.1
Changed lines of the file:
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@@
+	)
+	(junction
+		(at 119.38 185.42)
+		(diameter 0)
+		(color 0 0 0 0)
 	)
 	(junction
@@
 	)
 	(junction
+		(at 119.38 198.12)
+		(diameter 0)
+		(color 0 0 0 0)
+	)
+	(junction
 		(at 68.58 185.42)
 		(diameter 0)
@@
 	(wire
 		(pts
+			(xy 119.38 198.12) (xy 121.92 198.12)
+		)
+		(stroke
+			(width 0)
+			(type default)
+		)
+	)
+	(wire
+		(pts
 			(xy 101.6 170.18) (xy 80.01 170.18)
 		)
@@
 	(wire
 		(pts
-			(xy 105.41 185.42) (xy 121.92 185.42)
+			(xy 105.41 185.42) (xy 119.38 185.42)
 		)
 		(stroke
@@
 	(wire
 		(pts
+			(xy 119.38 185.42) (xy 121.92 185.42)
+		)
+		(stroke
+			(width 0)
+			(type default)
+		)
+	)
+	(wire
+		(pts
 			(xy 59.69 160.02) (xy 59.69 172.72)
 		)
@@
 	(wire
 		(pts
+			(xy 119.38 187.96) (xy 119.38 185.42)
+		)
+		(stroke
+			(width 0)
+			(type default)
+		)
+	)
+	(wire
+		(pts
 			(xy 35.56 123.19) (xy 39.37 123.19)
 		)
@@
 	(wire
 		(pts
-			(xy 106.68 198.12) (xy 121.92 198.12)
+			(xy 106.68 198.12) (xy 119.38 198.12)
 		)
 		(stroke
@@
 					(unit 1)
 				)
+			)
+		)
+	)
+	(symbol
+		(lib_id "easyeda2kicad:CC0402FRNPO9BN221")
+		(at 119.38 193.04 270)
+		(unit 1)
+		(exclude_from_sim no)
+		(in_bom yes)
+		(on_board yes)
+		(dnp no)
+		(property "Reference" "C136"
+			(at 123.19 193.04 0)
+			(effects
+				(font
+					(size 1.27 1.27)
+				)
+			)
+		)
+		(property "Value" "220pF"
+			(at 115.824 193.294 0)
+			(effects
+				(font
+					(size 1.27 1.27)
+				)
+			)
+		)
+		(property "Footprint" "easyeda2kicad:C0402"
+			(at 111.76 193.04 0)
+			(effects
+				(font
+					(size 1.27 1.27)
+				)
+				(hide yes)
+			)
+		)
+		(property "Datasheet" "https://lcsc.com/product-detail/Multilayer-Ceramic-Capacitors-MLCC-SMD-SMT_YAGEO-CC0402FRNPO9BN221_C326765.html"
+			(at 109.22 193.04 0)
+			(effects
+				(font
+					(size 1.27 1.27)
+				)
+				(hide yes)
+			)
+		)
+		(property "Description" "CC0402FRNPO9BN221"
+			(at 119.38 193.04 0)
+			(effects
+				(font
+					(size 1.27 1.27)
+				)
+				(hide yes)
+			)
+		)
+		(property "Manufacturer" "YAGEO(国巨)"
+			(at 106.68 193.04 0)
+			(effects
+				(font
+					(size 1.27 1.27)
+				)
+				(hide yes)
+			)
+		)
+		(property "MPN" "CC0402FRNPO9BN221"
+			(at 104.14 193.04 0)
+			(effects
+				(font
+					(size 1.27 1.27)
+				)
+				(hide yes)
+			)
+		)
+		(property "LCSC Part" "C326765"
+			(at 101.6 193.04 0)
+			(effects
+				(font
+					(size 1.27 1.27)
+				)
+				(hide yes)
+			)
+		)
+		(pin "1"
+		)
+		(pin "2"
+		)
+		(instances
+			(project ""
+				(path "/0c7b298e-2d07-4b1f-b033-e95f02d45089/4bf796fd-fdb4-45d1-808a-a634d5f4571e"
+					(reference "C136")
+					(unit 1)
+				)
