File: pcb/robot/USB-PD-ExtChg.kicad_sch (KiCad schematic)
At the start: 34 parts, among them J1 USBC_Receptacle_SMD_RA, Q3 AS2312, Q4 YJL3416A, U18 AP33771DKZ-13, U25 TVS0500DRV, U26 TPD1E05U06, U27 TPD1E05U06, U28 TPD1E05U06, U29 TPD1E05U06

Commit message: Modularized usb-pd board and main board split
Parts:
- renumbered D1 to D5, TP18 to TP22, TP18 to TP23, TP18 to TP9

Commit message: Re-unify USB-PD module into main board (single-PCB architecture) (#17)
Merges the USB-PD module circuitry back into the main robot board as
a single PCB, reversing the earlier main-board/USB-PD-daughter-board
split. Full re-route and re-placement of the combined design:

- Consolidated low-profile parts toward the board center, using the
  space freed up by relocated capacitors, for better overall use of
  the available area.
- Kept all 0-ohm test/isolation jumpers in accessible locations for
  bench testing.
- Added/corrected footprints for several parts that had broken or
  incorrect footprints (DDC6_TEX variants, SOT-23-6, SOT-23-3,
  R0402).

Carries forward every closed correction issue and update made since
the original split: #3 (CC jumpers), #6 (IC1.ON pull-down), #14/#15
(ADC divider, motor connector pinout), #16, #18 (I2C isolation
jumpers), #19 (charger-sense GPIO interrupt), plus the BOM/pricing
updates, LED changes, and MAX77642 replacement.

Verified via kicad-cli ERC/DRC + netlist diff against the pre-merge
board: 0 unconnected items (unchanged), no new DRC error-level
violations besides one pre-existing excluded item, and the #6
(IC1.ON pull-down) and #19 (charger-sense GPIO interrupt) circuits
confirmed intact at the net-topology level despite the full-board
re-annotation changing most reference designators. Most of the raw
diff size is a KiCad 9 footprint-format upgrade (pre-2023 format
rewritten to current) rather than design changes - spot-checked
against unrelated footprints (e.g. mounting holes), which show
identical geometry under the new syntax.
Parts:
- NT10: renamed from NT4; symbol Device:NetTie_2 -> robot:NetTie_2
- NT7: renamed from NT1; symbol Device:NetTie_2 -> robot:NetTie_2
- NT8: renamed from NT2; symbol Device:NetTie_2 -> robot:NetTie_2
- NT9: renamed from NT3; symbol Device:NetTie_2 -> robot:NetTie_2
- renumbered C18 to C26, C19 to C27, C20 to C28, C102 to C29, C103 to C30, C104 to C31, C105 to C32, D5 to D2, J1 to J3, Q3 to Q2, Q4 to Q3, R97 to R56, R51 to R57, R59 to R58, R58 to R59, R66 to R62, R62 to R63, R63 to R64, R64 to R65, TP22 to TP23, TP23 to TP24, TP9 to TP25, U28 to U15, U25 to U16, U26 to U17, U29 to U18, U27 to U19, U18 to U20
