File: pcb/robot/usb-pd-module/USB_PD_Module.kicad_sch (KiCad schematic)
At the start: 57 parts, among them J4 USB4151-GF-C, J9 Conn_01x16, U11 MAX77958EWV+T, U15 TPD1E05U06, U16 fpf1048bucx, U17 TPS61253AYFFT, U19 TPD1E05U06, U20 TPD1E05U06, U21 TPD1E05U06, U22 TPD1E05U06, U23 TPD1E05U06, U24 TVS0500DRV

Commit message: Update: Refreshed Gerbers and generated raw BOMs
I regenerated the motherboard gerbers, saved the modified footprints, and associated them with the schematic.
Parts:
- J9: now left out of the parts list
Changed lines of the file:
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@@
 		(unit 1)
 		(exclude_from_sim no)
-		(in_bom yes)
+		(in_bom no)
 		(on_board yes)
 		(dnp no)
@@
 			)
 		)
-		(property "Description" "Note this chip already has 22V Vbus to short (CC pins) protection so no external one required. "
+		(property "Description" "Note this chip already has 22V Vbus to short (CC pins) protection so no external one required."
 			(at 287.02 233.68 0)
 			(effects
