File: pcb/robot/usb-pd-module/USB_PD_Module.kicad_pcb (KiCad board)
At the start: 4 copper layers, 77 x 13.5 mm, 58 parts, among them J4 USB4151-GF-C, J9 Conn_01x16, U1 TPS22950CDDCR, U11 MAX77958EWV+T, U15 TPD1E05U06, U17 TPS61253AYFFT, U19 TPD1E05U06, U20 TPD1E05U06, U21 TPD1E05U06, U22 TPD1E05U06, U23 TPD1E05U06, U24 TVS0500DRV

Commit message: Add selectable 0-ohm CC jumpers on USB-PD module (addresses #3)
Insert R3 (CC1, populated) and R4 (CC2, DNP) in series between J4 and
the MAX77958 CC1/CC2 pins, so only one CC path is active for a direct
male USB-C plug configuration. Both jumpers placed in a separate area
with clear access for rework/probing.

Also cleaned up ERC findings found while editing: no-connect markers
on unused TPS22950CDDCR pin 6 and Conn_01x16 pin 5, and reorganized
power netclasses (Power_Module -> power_1A / Default).
Parts:
- added R3: 0, robot:R_0603_1608Metric, F.Cu at (131.5, 108.6)
- added R4: 0, robot:R_0603_1608Metric, F.Cu at (128.3, 108.6)
- moved U23 3.00 mm to (135.0, 110.5), turned to 180 degrees
- moved U21 2.40 mm to (133.4, 110.5), turned to 0 degrees
Connections:
- C45 pad 1: Net-(J4-CC2) -> Net-(U11-CC2)
- C46 pad 1: Net-(J4-CC1) -> Net-(U11-CC1)
- U11 pad A3: Net-(J4-CC1) -> Net-(U11-CC1)
- U11 pad A4: Net-(J4-CC2) -> Net-(U11-CC2)
Routing:
- net Net-(U11-CC2): track 0.00 -> 21.0 mm, vias 0 -> 2
- net Net-(J4-CC2): track 31.2 -> 13.9 mm, vias 4 -> 2
- net Net-(U11-CC1): track 0.00 -> 17.0 mm, vias 0 -> 2
- net Net-(J4-CC1): track 18.1 -> 12.3 mm, vias 4 -> 3
- net /AGND: track 75.3 -> 73.3 mm
- net Net-(J4-SBU1): track 11.4 -> 12.3 mm
- net GND: vias 52 -> 50
