File: pcb/robot/mcu/RP2040_minimal/RP2040_minimal.kicad_sch (KiCad schematic)
At the start: 42 parts, among them J2 Conn_01x05, U2 W25Q128JVS, U3 RP2040, Y1 ECS-120-8-36-CKM-TR3

Commit message: Replace ADC charger-sense front-end with GPIO interrupts (fixes #19)
Add 2x TPS3808G01DBVR voltage supervisors on USB_V and VRect
charger-sense paths, replacing the ADC divider+RC filter. GPIO26_ADC0/
GPIO27_ADC1 are now digital interrupt inputs (VIT~4.46V USB_V,
~2.11V VRect) instead of ADC channels.

Renamed net labels to reflect the digital nature of these signals:
ADC0 -> USB_SNS, ADC1 -> WLC_SNS (both hierarchical, crossing into
the MCU sheet), GPIO26_ADC0 -> GPIO26_USB_INT, GPIO27_ADC1 ->
GPIO27_WLC_INT (local labels). Documented the new circuit, threshold
derivation, and firmware implications in a schematic note replacing
the old #14-era one.

Verified via ERC/DRC against the pre-#19 baseline: 0 unconnected
items, no new error-level violations - only cosmetic silkscreen
warnings from the imported LCSC footprints.

Co-Authored-By: Claude Sonnet 5 <noreply@anthropic.com>
Parts:
- removed C39: 22nF, robot:C_0402_1005Metric, symbol robot:C
- added C35: 0.1uF, robot:C_0402_1005Metric, symbol robot:C
- added U14, U15: TPS3808G01DBVR, easyeda2kicad:SOT-23-6_L2.9-W1.6-P0.95-LS2.8-BR, symbol easyeda2kicad:TPS3808G01DBVR
- C38: value 22nF -> 0.1uF; Manufacturer Murata -> Samsung; Part Number GRM155R71H223KA12J -> CL05A104KA5NNNC; V_Max 50V -> (none)
- R24, R25: value 100 -> 100k; footprint robot:R_0603_1608Metric -> robot:R_0402_1005Metric; Manufacturer Stackpole Electronics -> UNI-ROYAL(Uniroyal Elec); Part Number RMCF0603JT100R -> 0402WGF1003TCE; Stock (none) -> 100
- R9: value 510k -> 422k; Manufacturer Stackpole Electronics -> YAGEO; Part Number RMCF0603JT510K -> RT0603BRD07422KL
Connections:
- net 3V3: now also C38.1, R24.1, R25.1, C35.1, U14.3 (MR), U14.6 (VDD), U15.3 (MR), U15.6 (VDD)
- net GND: now also C38.2, C35.2, U14.2 (GND), U15.2 (GND); no longer C38.1
- net at R12.1, R9.2: now also U15.5 (SENSE); no longer R24.2
- net ADC0 renamed GPIO27_WLC_INT
- net GPIO27_WLC_INT: now also U3.39 (GPIO27_ADC1), U15.1 (RESET)
- net ADC1 renamed WLC_SNS
- net GPIO26_ADC0 renamed GPIO26_USB_INT
- net GPIO26_USB_INT: now also R24.2, U14.1 (RESET); no longer R25.1
- removed net GPIO27_ADC1: C38.2, R24.1, U3.39 (GPIO27_ADC1)
- new net USB_SNS: U14.5 (SENSE)
- no-connect marks 1 -> 3
Other:
- note added: "TPS3808 voltage supervisors replace the passive divider+RC filter (fixes #19) - GPIO26_USB_INT/GPIO27_WLC_INT are now digital interrupt inputs, not ADC channels. Firmware: use GPIO input + edge interrupt, do not sample via ADC. U14/U15 = TPS3808G01DBVR (adjustable, SOT-23-6, LCSC C19653). SENSE vs internal 0.405V ref: VIT = (1+R1/R2) x 0.405V. MR->3V3 (unused). CT floating -> fixed 20ms delay. RE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"
- note removed: "LP Filter Corner @ 16 kHz."
- note removed: "New VRect sense divider (R9 510k / R12 100k), mirrors USB_V divider R16/R17. Gives ~3.28V at VRect=20V (TVS D10 SMF13A already bounds VRect below this). Not present before this revision - VRect used to feed the ADC front-end directly with no scaling/protection at all."
- note removed: "Protects analog inputs from overvolage on battery and charging monitoring pins"
- note removed: "SN74AHC125 removed - digital logic buffer cannot pass a proportional analog voltage (output saturates to rail based on VIH/VIL threshold, not the true input level). Replaced with passive high-impedance divider + RC filter, protected by RP2040's own internal clamp diodes (VPIN abs. max = IOVDD+0.5V per RP2040 datasheet 5.2.3.1). Fault current limited to <40uA by 510k/100k dividers (R16/R17, R9/R12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"
- moved on the sheet: C36, C37, R12, R22, R23, R9
