File: pcb/robot/mcu/RP2040_minimal/RP2040_minimal.kicad_sch (KiCad schematic)
At the start: 44 parts, among them J9 Conn_01x05, U24 W25Q128JVS, U29 RP2040, U30 TPS3808G01DBVR, U31 TPS3808G01DBVR, Y1 ECS-120-8-36-CKM-TR3

Commit message: Gate MAX77857 EN via GPIO22 divider, bump C136 to 100nF (#24)
R135/R136 (10k/10k) now gate U23.EN from GPIO22 instead of tying it
straight to 1.8V. GPIO22 low or floating (RP2040 reset/boot default)
holds EN at 0V, no firmware dependency for the off-state. VIO stays
on 1.8V, untouched. C136 220pF -> 100nF (CL05A104KA5NNNC) to meet
the MAX6006's real >=10nF minimum.

Verified against baseline: ERC 337/337 (no new violations), DRC 0
unconnected items, no violations tied to the new parts.
Connections:
- no-connect marks 3 -> 2
Changed lines of the file:
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@@
 		(at 367.03 260.35)
 	)
-	(no_connect
-		(at 254 167.64)
-	)
 	(wire
 		(pts
@@
 	(wire
 		(pts
-			(xy 231.14 167.64) (xy 254 167.64)
+			(xy 231.14 167.64) (xy 246.38 167.64)
 		)
 		(stroke
@@
 			(width 0)
 			(type default)
-		)
-	)
-	(label "GPIO22"
-		(at 254 167.64 180)
-		(effects
-			(font
-				(size 1.27 1.27)
-			)
-			(justify right bottom)
 		)
 	)
@@
 		(effects
 			(font
+				(size 1.27 1.27)
+			)
+			(justify left)
+		)
+	)
+	(hierarchical_label "GPIO22"
+		(shape input)
+		(at 246.38 167.64 0)
+		(effects
+			(font
